File: 40-channel HV switching board-p1.sch (KiCad schematic (older format))
At the start: 17 parts, among them J1 CONN_10, J2 CONN_50, J3 CONN_2, J4 CONN_2, SW1 4POS_SW, U16 PCA9505DGG

Commit message: Fix capcitor values on schematic, swap HV/GND on BNC jacks
Parts:
- C10, C11, C5: value 1uF -> 0.1uF
- C4: value 0.1uF -> 0.01uF
Changed lines of the file:
@@
-EESchema Schematic File Version 2  date 7/30/2011 2:04:39 PM
+EESchema Schematic File Version 2  date 11/18/2011 9:58:06 AM
 LIBS:power
 LIBS:device
@@
 Sheet 2 7
 Title "40-channel HV switching board"
-Date "30 jul 2011"
+Date "18 nov 2011"
 Rev "1"
 Comp "Ryan Fobel"
@@
 Comment4 ""
 $EndDescr
+Connection ~ 2050 3350
+Wire Wire Line
+	2050 3800 2050 3200
+Wire Wire Line
+	1950 3550 2150 3550
 Text GLabel 3000 6250 3    60   Input ~ 0
 A2
@@
 Wire Wire Line
 	1950 4000 1950 3550
-Connection ~ 2050 3350
 Wire Wire Line
 	2150 3800 2050 3800
-Wire Wire Line
-	2050 3800 2050 3200
 Connection ~ 4000 1000
 Wire Wire Line
@@
 Wire Wire Line
 	2050 3350 2150 3350
-Wire Wire Line
-	1950 3550 2150 3550
 Wire Wire Line
 	4400 4950 3550 4950
@@
 P 6800 4450
 F 0 "C11" H 6850 4550 50  0000 L CNN
-F 1 "1uF" H 6850 4350 50  0000 L CNN
+F 1 "0.1uF" H 6850 4350 50  0000 L CNN
 	1    6800 4450
 	1    0    0    -1
@@
 P 3550 5150
 F 0 "C10" H 3600 5250 50  0000 L CNN
-F 1 "1uF" H 3600 5050 50  0000 L CNN
+F 1 "0.1uF" H 3600 5050 50  0000 L CNN
 	1    3550 5150
 	1    0    0    -1
@@
 P 3650 1200
 F 0 "C4" H 3700 1300 50  0000 L CNN
-F 1 "0.1uF" H 3700 1100 50  0000 L CNN
+F 1 "0.01uF" H 3700 1100 50  0000 L CNN
 	1    3650 1200
 	1    0    0    -1
@@
 P 3300 1200
 F 0 "C5" H 3350 1300 50  0000 L CNN
-F 1 "1uF" H 3350 1100 50  0000 L CNN
+F 1 "0.1uF" H 3350 1100 50  0000 L CNN
 	1    3300 1200
 	1    0    0    -1
@@
 	1    0    0    -1
 $EndComp
-Text GLabel 1950 3550 0    60   Input ~ 0
+Text GLabel 1950 3200 0    60   Input ~ 0
 HVGND
 Text GLabel 6000 5850 2    60   Input ~ 0
@@
 Text GLabel 2100 1200 2    60   Input ~ 0
 SCL
-Text GLabel 1950 3200 0    60   Input ~ 0
+Text GLabel 1950 3550 0    60   Input ~ 0
 HV
 Text GLabel 9400 1750 0    60   Input ~ 0

Commit message: Update BOM for PCB assembly
Parts:
- R45: value 374 -> 375
Changed lines of the file:
@@
-EESchema Schematic File Version 2  date 11/18/2011 9:58:06 AM
+EESchema Schematic File Version 2  date 16/03/2012 12:06:03 AM
 LIBS:power
 LIBS:device
@@
 LIBS:valves
 LIBS:wheelerlab
-LIBS:40-channel HV switching board-cache
 EELAYER 25  0
 EELAYER END
@@
 Sheet 2 7
 Title "40-channel HV switching board"
-Date "18 nov 2011"
+Date "16 mar 2012"
 Rev "1"
 Comp "Ryan Fobel"
@@
 P 4000 1250
 F 0 "R45" V 4080 1250 50  0000 C CNN
-F 1 "374" V 4000 1250 50  0000 C CNN
+F 1 "375" V 4000 1250 50  0000 C CNN
 	1    4000 1250
 	1    0    0    -1

Commit message: Reindex channels to start at 0 instead of 1
This makes the hardware/software channel labels consistent.
Connections:
- net labels added: HVOUT0, OUT0
- net labels removed: HVOUT40, OUT40
Changed lines of the file:
@@
-EESchema Schematic File Version 2  date 16/03/2012 12:06:03 AM
+EESchema Schematic File Version 2  date 18/01/2013 10:50:53 AM
 LIBS:power
 LIBS:device
@@
 LIBS:valves
 LIBS:wheelerlab
+LIBS:40-channel HV switching board-cache
 EELAYER 25  0
 EELAYER END
@@
 Sheet 2 7
 Title "40-channel HV switching board"
-Date "16 mar 2012"
+Date "18 jan 2013"
 Rev "1"
 Comp "Ryan Fobel"
@@
 Text Notes 4800 2950 0    60   ~ 0
 40-CHANNEL GPIO
-Text Notes 8300 4350 0    60   ~ 0
+Text Notes 8300 4450 0    60   ~ 0
 TO DMF CHIP
 Text GLabel 9250 6650 0    60   Input ~ 0
@@
 +5V
 Text GLabel 6000 3850 2    60   Input ~ 0
+OUT36
+Text GLabel 6000 3650 2    60   Input ~ 0
 OUT37
-Text GLabel 6000 3650 2    60   Input ~ 0
+Text GLabel 6000 3550 2    60   Input ~ 0
 OUT38
-Text GLabel 6000 3550 2    60   Input ~ 0
+Text GLabel 6000 3450 2    60   Input ~ 0
 OUT39
-Text GLabel 6000 3450 2    60   Input ~ 0
-OUT40
 Text GLabel 6000 3950 2    60   Input ~ 0
-OUT36
+OUT35
 Text GLabel 6000 4050 2    60   Input ~ 0
-OUT35
+OUT34
 Text GLabel 6000 4150 2    60   Input ~ 0
-OUT34
+OUT33
 Text GLabel 6000 4350 2    60   Input ~ 0
-OUT33
+OUT32
 Text GLabel 6000 5250 2    60   Input ~ 0
+OUT24
+Text GLabel 6000 5150 2    60   Input ~ 0
 OUT25
-Text GLabel 6000 5150 2    60   Input ~ 0
+Text GLabel 6000 5050 2    60   Input ~ 0
 OUT26
-Text GLabel 6000 5050 2    60   Input ~ 0
+Text GLabel 6000 4850 2    60   Input ~ 0
 OUT27
-Text GLabel 6000 4850 2    60   Input ~ 0
+Text GLabel 6000 4450 2    60   Input ~ 0
+OUT31
+Text GLabel 6000 4550 2    60   Input ~ 0
+OUT30
+Text GLabel 6000 4650 2    60   Input ~ 0
+OUT29
+Text GLabel 6000 4750 2    60   Input ~ 0
 OUT28
-Text GLabel 6000 4450 2    60   Input ~ 0
-OUT32
-Text GLabel 6000 4550 2    60   Input ~ 0
-OUT31
-Text GLabel 6000 4650 2    60   Input ~ 0
-OUT30
-Text GLabel 6000 4750 2    60   Input ~ 0
-OUT29
 Text GLabel 6000 5750 2    60   Input ~ 0
+OUT20
+Text GLabel 6000 5650 2    60   Input ~ 0
 OUT21
-Text GLabel 6000 5650 2    60   Input ~ 0
+Text GLabel 6000 5550 2    60   Input ~ 0
 OUT22
-Text GLabel 6000 5550 2    60   Input ~ 0
+Text GLabel 6000 5350 2    60   Input ~ 0
 OUT23
-Text GLabel 6000 5350 2    60   Input ~ 0
-OUT24
 Text GLabel 4400 5750 0    60   Input ~ 0
-OUT20
+OUT19
 Text GLabel 4400 5650 0    60   Input ~ 0
-OUT19
+OUT18
 Text GLabel 4400 5550 0    60   Input ~ 0
-OUT18
+OUT17
 Text GLabel 4400 5350 0    60   Input ~ 0
-OUT17
+OUT16
 Text GLabel 4400 4850 0    60   Input ~ 0
+OUT12
+Text GLabel 4400 5050 0    60   Input ~ 0
 OUT13
-Text GLabel 4400 5050 0    60   Input ~ 0
+Text GLabel 4400 5150 0    60   Input ~ 0
 OUT14
-Text GLabel 4400 5150 0    60   Input ~ 0
+Text GLabel 4400 5250 0    60   Input ~ 0
 OUT15
-Text GLabel 4400 5250 0    60   Input ~ 0
-OUT16
 Text GLabel 4400 4750 0    60   Input ~ 0
-OUT12
+OUT11
 Text GLabel 4400 4650 0    60   Input ~ 0
-OUT11
+OUT10
 Text GLabel 4400 4550 0    60   Input ~ 0
-OUT10
+OUT9
 Text GLabel 4400 4450 0    60   Input ~ 0
-OUT9
+OUT8
 Text GLabel 4400 3450 0    60   Input ~ 0
+OUT0
+Text GLabel 4400 3550 0    60   Input ~ 0
 OUT1
-Text GLabel 4400 3550 0    60   Input ~ 0
+Text GLabel 4400 3650 0    60   Input ~ 0
 OUT2
-Text GLabel 4400 3650 0    60   Input ~ 0
+Text GLabel 4400 3850 0    60   Input ~ 0
 OUT3
-Text GLabel 4400 3850 0    60   Input ~ 0
+Text GLabel 4400 4350 0    60   Input ~ 0
+OUT7
+Text GLabel 4400 4150 0    60   Input ~ 0
+OUT6
+Text GLabel 4400 4050 0    60   Input ~ 0
+OUT5
+Text GLabel 4400 3950 0    60   Input ~ 0
 OUT4
-Text GLabel 4400 4350 0    60   Input ~ 0
-OUT8
-Text GLabel 4400 4150 0    60   Input ~ 0
-OUT7
-Text GLabel 4400 4050 0    60   Input ~ 0
-OUT6
-Text GLabel 4400 3950 0    60   Input ~ 0
-OUT5
 Text GLabel 4400 3350 0    60   Input ~ 0
 SCL
@@
 	1    0    0    -1
 $EndComp
+Text GLabel 9400 5250 0    60   Input ~ 0
+HVOUT35
+Text GLabel 9400 5350 0    60   Input ~ 0
+HVOUT36
+Text GLabel 9400 5550 0    60   Input ~ 0
+HVOUT38
+Text GLabel 9400 5450 0    60   Input ~ 0
+HVOUT37
+Text GLabel 9400 1750 0    60   Input ~ 0
+HVOUT0
+Text GLabel 9400 5650 0    60   Input ~ 0
+HVOUT39
 Text GLabel 9400 5150 0    60   Input ~ 0
-HVOUT35
-Text GLabel 9400 5250 0    60   Input ~ 0
-HVOUT36
-Text GLabel 9400 5450 0    60   Input ~ 0
-HVOUT38
-Text GLabel 9400 5350 0    60   Input ~ 0
-HVOUT37
-Text GLabel 9400 5650 0    60   Input ~ 0
-HVOUT40
-Text GLabel 9400 5550 0    60   Input ~ 0
-HVOUT39
+HVOUT34
 Text GLabel 9400 5050 0    60   Input ~ 0
-HVOUT34
+HVOUT33
+Text GLabel 9400 3450 0    60   Input ~ 0
+HVOUT17
+Text GLabel 9400 3550 0    60   Input ~ 0
+HVOUT18
+Text GLabel 9400 3750 0    60   Input ~ 0
+HVOUT20
+Text GLabel 9400 3650 0    60   Input ~ 0
+HVOUT19
+Text GLabel 9400 4050 0    60   Input ~ 0
+HVOUT23
+Text GLabel 9400 4150 0    60   Input ~ 0
+HVOUT24
+Text GLabel 9400 3950 0    60   Input ~ 0
+HVOUT22
+Text GLabel 9400 3850 0    60   Input ~ 0
+HVOUT21
+Text GLabel 9400 4650 0    60   Input ~ 0
+HVOUT29
+Text GLabel 9400 4750 0    60   Input ~ 0
+HVOUT30
 Text GLabel 9400 4950 0    60   Input ~ 0
-HVOUT33
+HVOUT32
+Text GLabel 9400 4850 0    60   Input ~ 0
+HVOUT31
+Text GLabel 9400 4450 0    60   Input ~ 0
+HVOUT27
+Text GLabel 9400 4550 0    60   Input ~ 0
+HVOUT28
+Text GLabel 9400 4350 0    60   Input ~ 0
+HVOUT26
+Text GLabel 9400 4250 0    60   Input ~ 0
+HVOUT25
+Text GLabel 9400 2650 0    60   Input ~ 0
+HVOUT9
+Text GLabel 9400 2750 0    60   Input ~ 0
+HVOUT10
+Text GLabel 9400 2950 0    60   Input ~ 0
+HVOUT12
+Text GLabel 9400 2850 0    60   Input ~ 0
+HVOUT11
+Text GLabel 9400 3250 0    60   Input ~ 0
+HVOUT15
 Text GLabel 9400 3350 0    60   Input ~ 0
-HVOUT17
-Text GLabel 9400 3450 0    60   Input ~ 0
-HVOUT18
-Text GLabel 9400 3650 0    60   Input ~ 0
-HVOUT20
-Text GLabel 9400 3550 0    60   Input ~ 0
-HVOUT19
-Text GLabel 9400 3950 0    60   Input ~ 0
-HVOUT23
-Text GLabel 9400 4050 0    60   Input ~ 0
-HVOUT24
-Text GLabel 9400 3850 0    60   Input ~ 0
-HVOUT22
-Text GLabel 9400 3750 0    60   Input ~ 0
-HVOUT21
-Text GLabel 9400 4550 0    60   Input ~ 0
-HVOUT29
-Text GLabel 9400 4650 0    60   Input ~ 0
-HVOUT30
-Text GLabel 9400 4850 0    60   Input ~ 0
-HVOUT32
-Text GLabel 9400 4750 0    60   Input ~ 0
-HVOUT31
-Text GLabel 9400 4350 0    60   Input ~ 0
-HVOUT27
-Text GLabel 9400 4450 0    60   Input ~ 0
-HVOUT28
-Text GLabel 9400 4250 0    60   Input ~ 0
-HVOUT26
-Text GLabel 9400 4150 0    60   Input ~ 0
-HVOUT25
+HVOUT16
+Text GLabel 9400 3150 0    60   Input ~ 0
+HVOUT14
+Text GLabel 9400 3050 0    60   Input ~ 0
+HVOUT13
+Text GLabel 9400 2250 0    60   Input ~ 0
+HVOUT5
+Text GLabel 9400 2350 0    60   Input ~ 0
+HVOUT6
 Text GLabel 9400 2550 0    60   Input ~ 0
-HVOUT9
-Text GLabel 9400 2650 0    60   Input ~ 0
-HVOUT10
-Text GLabel 9400 2850 0    60   Input ~ 0
-HVOUT12
-Text GLabel 9400 2750 0    60   Input ~ 0
-HVOUT11
-Text GLabel 9400 3150 0    60   Input ~ 0
-HVOUT15
-Text GLabel 9400 3250 0    60   Input ~ 0
-HVOUT16
-Text GLabel 9400 3050 0    60   Input ~ 0
-HVOUT14
-Text GLabel 9400 2950 0    60   Input ~ 0
-HVOUT13
+HVOUT8
+Text GLabel 9400 2450 0    60   Input ~ 0
+HVOUT7
+Text GLabel 9400 2050 0    60   Input ~ 0
+HVOUT3
 Text GLabel 9400 2150 0    60   Input ~ 0
-HVOUT5
-Text GLabel 9400 2250 0    60   Input ~ 0
-HVOUT6
-Text GLabel 9400 2450 0    60   Input ~ 0
-HVOUT8
-Text GLabel 9400 2350 0    60   Input ~ 0
-HVOUT7
+HVOUT4
 Text GLabel 9400 1950 0    60   Input ~ 0
-HVOUT3
-Text GLabel 9400 2050 0    60   Input ~ 0
-HVOUT4
-Text GLabel 9400 1850 0    60   Input ~ 0
 HVOUT2
 Text GLabel 2100 900  2    60   Input ~ 0
@@
 Text GLabel 1950 3550 0    60   Input ~ 0
 HV
-Text GLabel 9400 1750 0    60   Input ~ 0
+Text GLabel 9400 1850 0    60   Input ~ 0
 HVOUT1
 $Comp

Commit message: Replace 50-channel IDE connector with 40-channel
Parts:
- removed J2: CONN_50, symbol CONN_50
- added J2: CONN_40, symbol CONN_40
Connections:
- wire segments 52 -> 41
Changed lines of the file:
@@
-EESchema Schematic File Version 2  date 18/01/2013 10:50:53 AM
+EESchema Schematic File Version 2  date 18/01/2013 11:11:45 AM
 LIBS:power
 LIBS:device
@@
 LIBS:valves
 LIBS:wheelerlab
-LIBS:40-channel HV switching board-cache
 EELAYER 25  0
 EELAYER END
@@
 Comment4 ""
 $EndDescr
+$Comp
+L CONN_40 J2
+U 1 1 50F97415
+P 9650 3600
+F 0 "J2" V 9700 3600 60  0000 C CNN
+F 1 "CONN_40" V 9800 3600 60  0000 C CNN
+	1    9650 3600
+	1    0    0    -1
+$EndComp
 Connection ~ 2050 3350
 Wire Wire Line
@@
 Wire Wire Line
 	4400 5850 2150 5850
-Connection ~ 9250 5950
-Wire Wire Line
-	9400 5950 9250 5950
-Connection ~ 9250 6150
-Wire Wire Line
-	9400 6150 9250 6150
-Connection ~ 9250 6350
-Wire Wire Line
-	9400 6350 9250 6350
-Connection ~ 9250 6550
-Wire Wire Line
-	9400 6550 9250 6550
 Wire Wire Line
 	6800 4250 6000 4250
@@
 	6800 4950 6800 4650
 Wire Wire Line
-	9400 5750 9250 5750
-Wire Wire Line
-	9250 5750 9250 6650
-Wire Wire Line
-	9250 6650 9400 6650
-Wire Wire Line
-	9400 6450 9250 6450
-Connection ~ 9250 6450
-Wire Wire Line
-	9400 6250 9250 6250
-Connection ~ 9250 6250
-Wire Wire Line
-	9400 6050 9250 6050
-Connection ~ 9250 6050
-Wire Wire Line
-	9400 5850 9250 5850
-Connection ~ 9250 5850
-Wire Wire Line
 	2150 6050 4400 6050
 Wire Wire Line
@@
 Text Notes 8300 4450 0    60   ~ 0
 TO DMF CHIP
-Text GLabel 9250 6650 0    60   Input ~ 0
-HVGND
-$Comp
-L CONN_50 J2
-U 1 1 4E330420
-P 9650 4200
-F 0 "J2" V 9750 3800 60  0000 C CNN
-F 1 "CONN_50" V 9850 3800 60  0000 C CNN
-	1    9650 4200
-	1    0    0    -1
-$EndComp
 $Comp
 L C C11

Commit message: Use molex connector, fix BOM, ground planes, add logo
Parts:
- removed J1: CONN_10, symbol CONN_10
- removed R100, R43, R99: 4.75k, symbol R
- removed SW1: 4POS_SW, symbol 4POS_SW
- removed U16: PCA9505DGG, symbol PCA9505DGG
- added J1: CONN_4, symbol CONN_4
- added J2: CONN_10, symbol CONN_10
- added SW1: 12POS_SW, symbol 12POS_SW
- added U16: PCA9505/9506/9698, symbol PCA9505/9506/9698
- renumbered J2 to J5
Connections:
- wire segments 41 -> 46
- no-connect marks 3 -> 10
Other:
- note added: "COMMUNICATION\nBUS"
- note added: "POWER"
- note removed: "POWER AND\nCOMMUNICATION"
