File: 40-channel HV switching board-p1.sch (KiCad schematic (older format))
At the start: 15 parts, among them J1 CONN_4, J2 CONN_10, J3 CONN_2, J4 CONN_2, J5 CONN_40, SW1 12POS_SW, U16 PCA9505/9506/9698

Commit message: Reduce board footprint and replace GPIO
* Add ATMega328 chip and 74HC595s instead of GPIO
* Add jumpers to power MCU from USB and relays from VCC instead of PSU
* Com. bus should be capable of running at 5V or 3.3V
Parts:
- removed C4: 0.01uF, symbol C
- removed C9: 33uF, symbol CP1
- removed SW1: 12POS_SW, symbol 12POS_SW
- removed U16: PCA9505/9506/9698, symbol PCA9505/9506/9698
- added C1, C12, C13, C3, C6, C8, C9: 0.1uF, symbol C
- added C4: 33uF, symbol CP1
- added C7: 0.01uF, symbol C
- added IC1: ATMEG328PU, DIL28, symbol ATMEGA8-P
- added JP1, JP2: JUMPER, ~, symbol JUMPER
- added P1, P2: CONN_6, symbol CONN_6
- added R43: 10k, symbol R
- added R99: 1Meg, symbol R
- added SW1: DPST, symbol DPST
- added U1, U11, U16, U17, U6: 74HC595A, ~, symbol 74HC595A
- added X1: 16MHz, ~, symbol CRYSTAL
- C10, C11: value 0.1uF -> 22pF
Connections:
- net labels added: +5V_USB, MISO, MOSI, OE, RST, RX, SCK, SRCLR, SS, TX, VCC
- net labels removed: A0, A1, A2
- wire segments 46 -> 52
- no-connect marks 10 -> 19
Other:
- note added: "ARDUINO PROGRAMMING INTERFACE"
- note added: "ICSP"
- note added: "POWER JUMPERS"
- note added: "SHIFT REGISTERS"
- note removed: "40-CHANNEL GPIO"
- note removed: "I2C ADDRESS\nSELECTION"

Commit message: Add ISP latch circuit, use soft SPI
* replace 0603 caps with 1206
* label jumpers
* add LEDs for VCC, 5V, PROG MODE, and RESET
* move serial header to make it more accessible
Parts:
- added DS2, DS3, DS4: LED, symbol LED
- added JP3: JUMPER, ~, symbol JUMPER
- added R100, R125, R126, R127: 375, symbol R
- added U2: 4011, symbol 4011
Connections:
- net labels added: D7, S_MOSI, S_SCK, S_SS
- wire segments 52 -> 66
- no-connect marks 19 -> 11
Other:
- note added: "ISP LATCH"

Commit message: Modify ISP latch circuit, fix BOM
* Use 74LV00 NAND gate for ISP latch (3.3V compatible)
Parts:
- removed U2: 4011, symbol 4011
- added U6: 7400, ~, symbol 7400
- DS1: value LED -> +5V
- DS2: value LED -> VCC
- DS3: value LED -> PROG_MODE
- DS4: value LED -> RST
- renumbered U11 to U2, U17 to U3, U6 to U4, U16 to U5
Changed lines of the file:
@@
 Sheet 2 4
 Title ""
-Date "30 apr 2014"
+Date "5 may 2014"
 Rev ""
 Comp ""
@@
 P 2900 1650
 F 0 "DS1" H 2900 1750 50  0000 C CNN
-F 1 "LED" H 2900 1550 50  0000 C CNN
+F 1 "+5V" H 2900 1550 50  0000 C CNN
 F 2 "" H 2900 1650 60  0001 C CNN
 F 3 "" H 2900 1650 60  0001 C CNN
@@
 Wire Wire Line
 	3900 6750 4450 6750
-Text GLabel 850  5950 0    60   Input ~ 0
-+5V
 Text GLabel 850  6350 0    60   Input ~ 0
 GND
@@
 	1050 6350 1050 6050
 $Comp
-L 74HC595A U11
+L 74HC595A U2
 U 1 1 52EA8258
 P 4050 5600
-F 0 "U11" H 4200 6200 70  0000 C CNN
+F 0 "U2" H 4200 6200 70  0000 C CNN
 F 1 "74HC595A" H 4050 5000 70  0000 C CNN
 F 2 "~" H 4050 5600 60  0000 C CNN
@@
 	1    0    0    -1
 $EndComp
-Text GLabel 3150 5950 0    60   Input ~ 0
-+5V
 Text GLabel 3150 6350 0    60   Input ~ 0
 GND
@@
 	3350 5950 3150 5950
 $Comp
-L 74HC595A U17
+L 74HC595A U3
 U 1 1 52EA8268
 P 6400 5600
-F 0 "U17" H 6550 6200 70  0000 C CNN
+F 0 "U3" H 6550 6200 70  0000 C CNN
 F 1 "74HC595A" H 6400 5000 70  0000 C CNN
 F 2 "~" H 6400 5600 60  0000 C CNN
@@
 	5700 6350 5700 6050
 $Comp
-L 74HC595A U6
+L 74HC595A U4
 U 1 1 52EA8362
 P 2800 7200
-F 0 "U6" H 2950 7800 70  0000 C CNN
+F 0 "U4" H 2950 7800 70  0000 C CNN
 F 1 "74HC595A" H 2800 6600 70  0000 C CNN
 F 2 "~" H 2800 7200 60  0000 C CNN
@@
 Wire Wire Line
 	1950 7550 2100 7550
-Text GLabel 5500 5950 0    60   Input ~ 0
-+5V
-Text GLabel 1950 7550 0    60   Input ~ 0
-+5V
 Text GLabel 1950 7950 0    60   Input ~ 0
 GND
@@
 	2100 6500 2100 6750
 $Comp
-L 74HC595A U16
+L 74HC595A U5
 U 1 1 52EA8645
 P 5150 7200
-F 0 "U16" H 5300 7800 70  0000 C CNN
+F 0 "U5" H 5300 7800 70  0000 C CNN
 F 1 "74HC595A" H 5150 6600 70  0000 C CNN
 F 2 "~" H 5150 7200 60  0000 C CNN
@@
 	1    0    0    -1
 $EndComp
-Text GLabel 4300 7550 0    60   Input ~ 0
-+5V
 Text GLabel 4300 7950 0    60   Input ~ 0
 GND
@@
 Text GLabel 1150 2700 2    60   Input ~ 0
 SCK
-$Comp
-L 4011 U2
-U 1 1 536131ED
-P 4500 2900
-F 0 "U2" H 4500 2950 60  0000 C CNN
-F 1 "4011" H 4500 2850 60  0000 C CNN
-F 2 "" H 4500 2900 60  0000 C CNN
-F 3 "" H 4500 2900 60  0000 C CNN
-	1    4500 2900
-	1    0    0    -1
-$EndComp
-$Comp
-L 4011 U2
-U 2 1 53613264
-P 4500 2350
-F 0 "U2" H 4500 2400 60  0000 C CNN
-F 1 "4011" H 4500 2300 60  0000 C CNN
-F 2 "" H 4500 2350 60  0000 C CNN
-F 3 "" H 4500 2350 60  0000 C CNN
-	2    4500 2350
-	1    0    0    -1
-$EndComp
-$Comp
-L 4011 U2
-U 3 1 53613284
-P 4500 3550
-F 0 "U2" H 4500 3600 60  0000 C CNN
-F 1 "4011" H 4500 3500 60  0000 C CNN
-F 2 "" H 4500 3550 60  0000 C CNN
-F 3 "" H 4500 3550 60  0000 C CNN
-	3    4500 3550
-	1    0    0    -1
-$EndComp
-$Comp
-L 4011 U2
-U 4 1 53613299
-P 5750 3250
-F 0 "U2" H 5750 3300 60  0000 C CNN
-F 1 "4011" H 5750 3200 60  0000 C CNN
-F 2 "" H 5750 3250 60  0000 C CNN
-F 3 "" H 5750 3250 60  0000 C CNN
-	4    5750 3250
-	1    0    0    -1
-$EndComp
 Text GLabel 3900 3450 0    60   Input ~ 0
 SDA
 Text GLabel 3900 3650 0    60   Input ~ 0
-+5V
+VCC
 Text GLabel 4300 1950 0    60   Input ~ 0
-+5V
+VCC
 Wire Wire Line
 	4300 1950 4300 2150
@@
 $EndComp
 Text GLabel 3650 2500 0    60   Input ~ 0
-+5V
+VCC
 Wire Wire Line
 	3650 3000 3900 3000
@@
 U 1 1 53613CEC
 P 5100 2150
-F 0 "DS3" H 5100 2250 50  0000 C CNN
-F 1 "LED" H 5100 2050 50  0000 C CNN
+F 0 "DS3" H 5100 2050 50  0000 C CNN
+F 1 "PROG_MODE" H 5100 2250 50  0000 C CNN
 F 2 "" H 5100 2150 60  0001 C CNN
 F 3 "" H 5100 2150 60  0001 C CNN
@@
 P 6350 3050
 F 0 "DS4" H 6350 3150 50  0000 C CNN
-F 1 "LED" H 6350 2950 50  0000 C CNN
+F 1 "RST" H 6350 2950 50  0000 C CNN
 F 2 "" H 6350 3050 60  0001 C CNN
 F 3 "" H 6350 3050 60  0001 C CNN
@@
 $EndComp
 Text GLabel 5850 2850 0    60   Input ~ 0
-+5V
+VCC
 Wire Wire Line
 	4300 1950 4600 1950
@@
 P 3600 1650
 F 0 "DS2" H 3600 1750 50  0000 C CNN
-F 1 "LED" H 3600 1550 50  0000 C CNN
+F 1 "VCC" H 3600 1550 50  0000 C CNN
 F 2 "" H 3600 1650 60  0001 C CNN
 F 3 "" H 3600 1650 60  0001 C CNN
@@
 Text GLabel 8700 750  2    60   Input ~ 0
 GND
+$Comp
+L 7400 U6
+U 1 1 5363FEF8
+P 4500 2900
+F 0 "U6" H 4500 2950 60  0000 C CNN
+F 1 "7400" H 4500 2800 60  0000 C CNN
+F 2 "~" H 4500 2900 60  0000 C CNN
+F 3 "~" H 4500 2900 60  0000 C CNN
+	1    4500 2900
+	1    0    0    -1
+$EndComp
+$Comp
+L 7400 U6
+U 2 1 5363FF1E
+P 4500 2350
+F 0 "U6" H 4500 2400 60  0000 C CNN
+F 1 "7400" H 4500 2250 60  0000 C CNN
+F 2 "~" H 4500 2350 60  0000 C CNN
+F 3 "~" H 4500 2350 60  0000 C CNN
+	2    4500 2350
+	1    0    0    -1
+$EndComp
+$Comp
+L 7400 U6
+U 3 1 53640100
+P 4500 3550
+F 0 "U6" H 4500 3600 60  0000 C CNN
+F 1 "7400" H 4500 3450 60  0000 C CNN
+F 2 "~" H 4500 3550 60  0000 C CNN
+F 3 "~" H 4500 3550 60  0000 C CNN
+	3    4500 3550
+	1    0    0    -1
+$EndComp
+$Comp
+L 7400 U6
+U 4 1 5364010B
+P 5750 3250
+F 0 "U6" H 5750 3300 60  0000 C CNN
+F 1 "7400" H 5750 3150 60  0000 C CNN
+F 2 "~" H 5750 3250 60  0000 C CNN
+F 3 "~" H 5750 3250 60  0000 C CNN
+	4    5750 3250
+	1    0    0    -1
+$EndComp
+Text GLabel 4300 7550 0    60   Input ~ 0
++5V
+Text GLabel 1950 7550 0    60   Input ~ 0
++5V
+Text GLabel 5500 5950 0    60   Input ~ 0
++5V
+Text GLabel 3150 5950 0    60   Input ~ 0
++5V
+Text GLabel 850  5950 0    60   Input ~ 0
++5V
 $EndSCHEMATC

Commit message: Make LED current-limiting resistors 1k
Parts:
- R100, R125, R126, R127, R45: value 375 -> 1k
Changed lines of the file:
@@
 P 2900 1200
 F 0 "R45" V 2980 1200 50  0000 C CNN
-F 1 "375" V 2900 1200 50  0000 C CNN
+F 1 "1k" V 2900 1200 50  0000 C CNN
 F 2 "" H 2900 1200 60  0001 C CNN
 F 3 "" H 2900 1200 60  0001 C CNN
@@
 P 3650 2750
 F 0 "R100" V 3730 2750 50  0000 C CNN
-F 1 "375" V 3650 2750 50  0000 C CNN
+F 1 "1k" V 3650 2750 50  0000 C CNN
 F 2 "" H 3650 2750 60  0001 C CNN
 F 3 "" H 3650 2750 60  0001 C CNN
@@
 P 4850 1950
 F 0 "R125" V 4930 1950 50  0000 C CNN
-F 1 "375" V 4850 1950 50  0000 C CNN
+F 1 "1k" V 4850 1950 50  0000 C CNN
 F 2 "" H 4850 1950 60  0001 C CNN
 F 3 "" H 4850 1950 60  0001 C CNN
@@
 P 6100 2850
 F 0 "R126" V 6180 2850 50  0000 C CNN
-F 1 "375" V 6100 2850 50  0000 C CNN
+F 1 "1k" V 6100 2850 50  0000 C CNN
 F 2 "" H 6100 2850 60  0001 C CNN
 F 3 "" H 6100 2850 60  0001 C CNN
@@
 P 3600 1200
 F 0 "R127" V 3680 1200 50  0000 C CNN
-F 1 "375" V 3600 1200 50  0000 C CNN
+F 1 "1k" V 3600 1200 50  0000 C CNN
 F 2 "" H 3600 1200 60  0001 C CNN
 F 3 "" H 3600 1200 60  0001 C CNN

Commit message: Add decoupling capacitor to 7400 chip, label LED polarity
Parts:
- added C14: 0.1uF, symbol C
Connections:
- wire segments 66 -> 65
Other:
- note added: "ISP"
- note removed: "ICSP"
Changed lines of the file:
@@
 EELAYER 27 0
 EELAYER END
-$Descr User 11000 8500
+$Descr USLetter 11000 8500
 encoding utf-8
 Sheet 2 4
-Title ""
-Date "5 may 2014"
-Rev ""
-Comp ""
+Title "40-channel HV switching board"
+Date "6 may 2014"
+Rev "2.1"
+Comp "Ryan Fobel"
 Comment1 ""
 Comment2 ""
@@
 Connection ~ 1500 950
 Connection ~ 2200 950
-Wire Wire Line
-	2900 950  2900 800
 Connection ~ 2900 950
 Wire Wire Line
@@
 L CONN_40 J5
 U 1 1 52E82584
-P 10150 5150
-F 0 "J5" V 10200 5150 60  0000 C CNN
-F 1 "CONN_40" V 10300 5150 60  0000 C CNN
-F 2 "" H 10150 5150 60  0001 C CNN
-F 3 "" H 10150 5150 60  0001 C CNN
-	1    10150 5150
+P 10150 5250
+F 0 "J5" V 10200 5250 60  0000 C CNN
+F 1 "CONN_40" V 10300 5250 60  0000 C CNN
+F 2 "" H 10150 5250 60  0001 C CNN
+F 3 "" H 10150 5250 60  0001 C CNN
+	1    10150 5250
 	1    0    0    -1
 $EndComp
@@
 Text Notes 4200 4900 0    60   ~ 0
 SHIFT REGISTERS
-Text Notes 9650 7400 0    60   ~ 0
+Text Notes 9800 3300 0    60   ~ 0
 TO DMF CHIP
 Text GLabel 2900 1850 2    60   Input ~ 0
@@
 Text GLabel 2900 950  2    60   Input ~ 0
 +5V
-$Comp
-L +5V #PWR01
-U 1 1 52E82587
-P 2900 800
-F 0 "#PWR01" H 2900 890 20  0001 C CNN
-F 1 "+5V" H 2900 890 30  0000 C CNN
-F 2 "" H 2900 800 60  0001 C CNN
-F 3 "" H 2900 800 60  0001 C CNN
-	1    2900 800
-	1    0    0    -1
-$EndComp
 Text Notes 700  850  0    60   ~ 0
 POWER
@@
 Text GLabel 1900 2000 0    60   Input ~ 0
 HVGND
+Text GLabel 9900 6900 0    60   Input ~ 0
+HVOUT35
+Text GLabel 9900 7000 0    60   Input ~ 0
+HVOUT36
+Text GLabel 9900 7200 0    60   Input ~ 0
+HVOUT38
+Text GLabel 9900 7100 0    60   Input ~ 0
+HVOUT37
+Text GLabel 9900 3400 0    60   Input ~ 0
+HVOUT0
+Text GLabel 9900 7300 0    60   Input ~ 0
+HVOUT39
 Text GLabel 9900 6800 0    60   Input ~ 0
-HVOUT35
-Text GLabel 9900 6900 0    60   Input ~ 0
-HVOUT36
-Text GLabel 9900 7100 0    60   Input ~ 0
-HVOUT38
-Text GLabel 9900 7000 0    60   Input ~ 0
-HVOUT37
-Text GLabel 9900 3300 0    60   Input ~ 0
-HVOUT0
-Text GLabel 9900 7200 0    60   Input ~ 0
-HVOUT39
+HVOUT34
 Text GLabel 9900 6700 0    60   Input ~ 0
-HVOUT34
+HVOUT33
+Text GLabel 9900 5100 0    60   Input ~ 0
+HVOUT17
+Text GLabel 9900 5200 0    60   Input ~ 0
+HVOUT18
+Text GLabel 9900 5400 0    60   Input ~ 0
+HVOUT20
+Text GLabel 9900 5300 0    60   Input ~ 0
+HVOUT19
+Text GLabel 9900 5700 0    60   Input ~ 0
+HVOUT23
+Text GLabel 9900 5800 0    60   Input ~ 0
+HVOUT24
+Text GLabel 9900 5600 0    60   Input ~ 0
+HVOUT22
+Text GLabel 9900 5500 0    60   Input ~ 0
+HVOUT21
+Text GLabel 9900 6300 0    60   Input ~ 0
+HVOUT29
+Text GLabel 9900 6400 0    60   Input ~ 0
+HVOUT30
 Text GLabel 9900 6600 0    60   Input ~ 0
-HVOUT33
+HVOUT32
+Text GLabel 9900 6500 0    60   Input ~ 0
+HVOUT31
+Text GLabel 9900 6100 0    60   Input ~ 0
+HVOUT27
+Text GLabel 9900 6200 0    60   Input ~ 0
+HVOUT28
+Text GLabel 9900 6000 0    60   Input ~ 0
+HVOUT26
+Text GLabel 9900 5900 0    60   Input ~ 0
+HVOUT25
+Text GLabel 9900 4300 0    60   Input ~ 0
+HVOUT9
+Text GLabel 9900 4400 0    60   Input ~ 0
+HVOUT10
+Text GLabel 9900 4600 0    60   Input ~ 0
+HVOUT12
+Text GLabel 9900 4500 0    60   Input ~ 0
+HVOUT11
+Text GLabel 9900 4900 0    60   Input ~ 0
+HVOUT15
 Text GLabel 9900 5000 0    60   Input ~ 0
-HVOUT17
-Text GLabel 9900 5100 0    60   Input ~ 0
-HVOUT18
-Text GLabel 9900 5300 0    60   Input ~ 0
-HVOUT20
-Text GLabel 9900 5200 0    60   Input ~ 0
-HVOUT19
-Text GLabel 9900 5600 0    60   Input ~ 0
-HVOUT23
-Text GLabel 9900 5700 0    60   Input ~ 0
-HVOUT24
-Text GLabel 9900 5500 0    60   Input ~ 0
-HVOUT22
-Text GLabel 9900 5400 0    60   Input ~ 0
-HVOUT21
-Text GLabel 9900 6200 0    60   Input ~ 0
-HVOUT29
-Text GLabel 9900 6300 0    60   Input ~ 0
-HVOUT30
-Text GLabel 9900 6500 0    60   Input ~ 0
-HVOUT32
-Text GLabel 9900 6400 0    60   Input ~ 0
-HVOUT31
-Text GLabel 9900 6000 0    60   Input ~ 0
-HVOUT27
-Text GLabel 9900 6100 0    60   Input ~ 0
-HVOUT28
-Text GLabel 9900 5900 0    60   Input ~ 0
-HVOUT26
-Text GLabel 9900 5800 0    60   Input ~ 0
-HVOUT25
+HVOUT16
+Text GLabel 9900 4800 0    60   Input ~ 0
+HVOUT14
+Text GLabel 9900 4700 0    60   Input ~ 0
+HVOUT13
+Text GLabel 9900 3900 0    60   Input ~ 0
+HVOUT5
+Text GLabel 9900 4000 0    60   Input ~ 0
+HVOUT6
 Text GLabel 9900 4200 0    60   Input ~ 0
-HVOUT9
-Text GLabel 9900 4300 0    60   Input ~ 0
-HVOUT10
-Text GLabel 9900 4500 0    60   Input ~ 0
-HVOUT12
-Text GLabel 9900 4400 0    60   Input ~ 0
-HVOUT11
-Text GLabel 9900 4800 0    60   Input ~ 0
-HVOUT15
-Text GLabel 9900 4900 0    60   Input ~ 0
-HVOUT16
-Text GLabel 9900 4700 0    60   Input ~ 0
-HVOUT14
-Text GLabel 9900 4600 0    60   Input ~ 0
-HVOUT13
+HVOUT8
+Text GLabel 9900 4100 0    60   Input ~ 0
+HVOUT7
+Text GLabel 9900 3700 0    60   Input ~ 0
+HVOUT3
 Text GLabel 9900 3800 0    60   Input ~ 0
-HVOUT5
-Text GLabel 9900 3900 0    60   Input ~ 0
-HVOUT6
-Text GLabel 9900 4100 0    60   Input ~ 0
-HVOUT8
-Text GLabel 9900 4000 0    60   Input ~ 0
-HVOUT7
+HVOUT4
 Text GLabel 9900 3600 0    60   Input ~ 0
-HVOUT3
-Text GLabel 9900 3700 0    60   Input ~ 0
-HVOUT4
-Text GLabel 9900 3500 0    60   Input ~ 0
 HVOUT2
 Text GLabel 1150 2100 2    60   Input ~ 0
@@
 Text GLabel 1900 2350 0    60   Input ~ 0
 HV
-Text GLabel 9900 3400 0    60   Input ~ 0
+Text GLabel 9900 3500 0    60   Input ~ 0
 HVOUT1
 $Comp
@@
 GND
 Text Notes 8050 6500 0    60   ~ 0
-ICSP
+ISP
 Text GLabel 9300 2850 2    60   Input ~ 0
 S_SCK
@@
 Text GLabel 6950 3250 2    60   Input ~ 0
 RST
-Text Notes 4300 1800 0    60   ~ 0
+Text Notes 4650 1600 0    60   ~ 0
 ISP LATCH
 $Comp
@@
 Text GLabel 850  5950 0    60   Input ~ 0
 +5V
+$Comp
+L C C14
+U 1 1 5367B80F
+P 4300 1750
+F 0 "C14" H 4350 1850 50  0000 L CNN
+F 1 "0.1uF" H 4050 1650 50  0000 L CNN
+F 2 "" H 4300 1750 60  0001 C CNN
+F 3 "" H 4300 1750 60  0001 C CNN
+	1    4300 1750
+	1    0    0    -1
+$EndComp
+Text GLabel 4300 1550 2    60   Input ~ 0
+GND
 $EndSCHEMATC
