File: 40-channel HV switching board-p2.sch (KiCad schematic (older format))
At the start: 34 parts, among them U1 74AC540, U2 AQW216, U27 AQW216, U28 AQW216, U29 AQW216, U3 AQW216, U30 AQW216, U4 AQW216, U5 AQW216

Commit message: Fix capcitor values on schematic, swap HV/GND on BNC jacks
Parts:
- C1: value 1uF -> 0.1uF
Changed lines of the file:
@@
-EESchema Schematic File Version 2  date 7/30/2011 2:04:39 PM
+EESchema Schematic File Version 2  date 11/18/2011 9:58:06 AM
 LIBS:power
 LIBS:device
@@
 Sheet 3 7
 Title "40-channel HV switching board"
-Date "30 jul 2011"
+Date "18 nov 2011"
 Rev "1"
 Comp "Ryan Fobel"
@@
 P 3700 1150
 F 0 "C1" H 3600 1250 50  0000 L CNN
-F 1 "1uF" H 3550 1050 50  0000 L CNN
+F 1 "0.1uF" H 3500 1050 50  0000 L CNN
 	1    3700 1150
 	0    1    1    0

Commit message: Reindex channels to start at 0 instead of 1
This makes the hardware/software channel labels consistent.
Connections:
- net labels added: HVOUT0, OUT0
- net labels removed: HVOUT8, OUT8
Changed lines of the file:
@@
-EESchema Schematic File Version 2  date 16/03/2012 12:06:03 AM
+EESchema Schematic File Version 2  date 18/01/2013 10:50:53 AM
 LIBS:power
 LIBS:device
@@
 LIBS:valves
 LIBS:wheelerlab
+LIBS:40-channel HV switching board-cache
 EELAYER 25  0
 EELAYER END
@@
 Sheet 3 7
 Title "40-channel HV switching board"
-Date "16 mar 2012"
+Date "18 jan 2013"
 Rev "1"
 Comp "Ryan Fobel"
@@
 	950  4150 5450 4150
 Text GLabel 1100 2100 0    60   Input ~ 0
-OUT5
+OUT4
 $Comp
 L R R67
@@
 $EndComp
 Text GLabel 3000 7100 2    60   Input ~ 0
-HVOUT8
+HVOUT7
 Text GLabel 3000 7350 2    60   Input ~ 0
 HV
@@
 $EndComp
 Text GLabel 2050 7350 0    60   Input ~ 0
-OUT8
+OUT7
 Text GLabel 2050 6150 0    60   Input ~ 0
-OUT7
+OUT6
 $Comp
 L +5V #PWR06
@@
 HV
 Text GLabel 3000 5900 2    60   Input ~ 0
-HVOUT7
+HVOUT6
 $Comp
 L R R2
@@
 $EndComp
 Text GLabel 5850 5900 2    60   Input ~ 0
-HVOUT5
+HVOUT4
 Text GLabel 5850 6150 2    60   Input ~ 0
 HV
@@
 $EndComp
 Text GLabel 4900 6150 0    60   Input ~ 0
+OUT4
+Text GLabel 4900 7350 0    60   Input ~ 0
 OUT5
-Text GLabel 4900 7350 0    60   Input ~ 0
-OUT6
 $Comp
 L +5V #PWR08
@@
 HV
 Text GLabel 5850 7100 2    60   Input ~ 0
-HVOUT6
+HVOUT5
 $Comp
 L R R66
@@
 $EndComp
 Text GLabel 9550 4000 2    60   Input ~ 0
-HVOUT3
+HVOUT2
 Text GLabel 9550 4250 2    60   Input ~ 0
 HV
@@
 $EndComp
 Text GLabel 8600 4250 0    60   Input ~ 0
+OUT2
+Text GLabel 8600 5450 0    60   Input ~ 0
 OUT3
-Text GLabel 8600 5450 0    60   Input ~ 0
-OUT4
 $Comp
 L +5V #PWR010
@@
 HV
 Text GLabel 9550 5200 2    60   Input ~ 0
-HVOUT4
+HVOUT3
 $Comp
 L R R65
@@
 $EndComp
 Text GLabel 9550 2750 2    60   Input ~ 0
-HVOUT2
+HVOUT1
 Text GLabel 9550 3000 2    60   Input ~ 0
 HV
@@
 $EndComp
 Text GLabel 8600 3000 0    60   Input ~ 0
-OUT2
+OUT1
 Text GLabel 8600 1800 0    60   Input ~ 0
-OUT1
+OUT0
 Text GLabel 1100 1700 0    60   Input ~ 0
-OUT1
+OUT0
 $Comp
 L 74AC540 U1
@@
 $EndComp
 Text GLabel 1100 2700 0    60   Input ~ 0
+OUT5
+Text GLabel 1100 2500 0    60   Input ~ 0
+OUT7
+Text GLabel 1100 2300 0    60   Input ~ 0
 OUT6
-Text GLabel 1100 2500 0    60   Input ~ 0
-OUT8
-Text GLabel 1100 2300 0    60   Input ~ 0
-OUT7
 Text GLabel 1100 1900 0    60   Input ~ 0
+OUT2
+Text GLabel 1100 2900 0    60   Input ~ 0
 OUT3
-Text GLabel 1100 2900 0    60   Input ~ 0
-OUT4
 Text GLabel 1100 3100 0    60   Input ~ 0
-OUT2
+OUT1
 $Comp
 L GND #PWR013
@@
 HV
 Text GLabel 9550 1550 2    60   Input ~ 0
-HVOUT1
+HVOUT0
 $Comp
 L R R5
