File: 40-channel HV switching board-p2.sch (KiCad schematic (older format))
At the start: 34 parts, among them U1 74AC540, U2 AQW216, U27 AQW216, U28 AQW216, U29 AQW216, U3 AQW216, U30 AQW216, U4 AQW216, U5 AQW216

Commit message: Reroute onto 2-layer board, remove inverters
Parts:
- removed C1: 0.1uF, symbol C
- removed U1: 74AC540, symbol 74AC540
- added R13, R18, R19, R24, R25, R36, R75, R80, R81, R86, R87, R98: 4.75k, symbol R
- added R14, R15, R16, R17, R20, R21, R22, R23, R28, R29, R34, R35, R76, R77, R78, R79, R82, R83, R84, R85, R88, R89, R94, R95: 375, symbol R
- added U10, U14, U15, U31, U32, U33, U34, U35, U36, U7, U8, U9: AQW216, symbol AQW216
Connections:
- net labels added: HVOUT10, HVOUT11, HVOUT12, HVOUT13, HVOUT14, HVOUT15, HVOUT16, HVOUT17, HVOUT18, HVOUT19, HVOUT8, HVOUT9, OUT10, OUT11, OUT12, OUT13, OUT14, OUT15, OUT16, OUT17, OUT18, OUT19, OUT8, OUT9
- wire segments 142 -> 140

Commit message: Rename PhotoMOS reference numbers to match channel number
Parts:
- renumbered U5 to CH0, U27 to CH1, U9 to CH10, U32 to CH11, U8 to CH12, U33 to CH13, U7 to CH14, U34 to CH15, U15 to CH16, U35 to CH17, U14 to CH18, U36 to CH19, U4 to CH2, U28 to CH3, U3 to CH4, U29 to CH5, U2 to CH6, U30 to CH7, U10 to CH8, U31 to CH9
Changed lines of the file:
@@
 LIBS:valves
 LIBS:wheelerlab
+LIBS:40-channel HV switching board-cache
 EELAYER 27 0
 EELAYER END
@@
 Sheet 3 4
 Title "40-channel HV switching board"
-Date "4 feb 2014"
+Date "30 apr 2014"
 Rev "1"
 Comp "Ryan Fobel"
@@
 $EndComp
 $Comp
-L AQW216 U30
+L AQW216 CH7
 U 1 1 52E6DB5D
 P 1800 7500
-F 0 "U30" H 1800 7850 60  0000 C CNN
+F 0 "CH7" H 1800 7850 60  0000 C CNN
 F 1 "AQW216" H 1800 7145 60  0000 C CNN
 F 2 "" H 1800 7500 60  0001 C CNN
@@
 $EndComp
 $Comp
-L AQW216 U2
+L AQW216 CH6
 U 1 1 52E6D491
 P 1800 6600
-F 0 "U2" H 1800 6950 60  0000 C CNN
+F 0 "CH6" H 1800 6950 60  0000 C CNN
 F 1 "AQW216" H 1800 6245 60  0000 C CNN
 F 2 "" H 1800 6600 60  0001 C CNN
@@
 $EndComp
 $Comp
-L AQW216 U3
+L AQW216 CH4
 U 1 1 52E6D494
 P 1800 4800
-F 0 "U3" H 1800 5150 60  0000 C CNN
+F 0 "CH4" H 1800 5150 60  0000 C CNN
 F 1 "AQW216" H 1800 4445 60  0000 C CNN
 F 2 "" H 1800 4800 60  0001 C CNN
@@
 $EndComp
 $Comp
-L AQW216 U29
+L AQW216 CH5
 U 1 1 52E6D497
 P 1800 5700
-F 0 "U29" H 1800 6050 60  0000 C CNN
+F 0 "CH5" H 1800 6050 60  0000 C CNN
 F 1 "AQW216" H 1800 5345 60  0000 C CNN
 F 2 "" H 1800 5700 60  0001 C CNN
@@
 $EndComp
 $Comp
-L AQW216 U4
+L AQW216 CH2
 U 1 1 52E6DB69
 P 1800 3000
-F 0 "U4" H 1800 3350 60  0000 C CNN
+F 0 "CH2" H 1800 3350 60  0000 C CNN
 F 1 "AQW216" H 1800 2645 60  0000 C CNN
 F 2 "" H 1800 3000 60  0001 C CNN
@@
 $EndComp
 $Comp
-L AQW216 U28
+L AQW216 CH3
 U 1 1 52E6DB6C
 P 1800 3900
-F 0 "U28" H 1800 4250 60  0000 C CNN
+F 0 "CH3" H 1800 4250 60  0000 C CNN
 F 1 "AQW216" H 1800 3545 60  0000 C CNN
 F 2 "" H 1800 3900 60  0001 C CNN
@@
 HVGND
 $Comp
-L AQW216 U5
+L AQW216 CH0
 U 1 1 52E6DB73
 P 1800 1200
-F 0 "U5" H 1800 1550 60  0000 C CNN
+F 0 "CH0" H 1800 1550 60  0000 C CNN
 F 1 "AQW216" H 1800 845 60  0000 C CNN
 F 2 "" H 1800 1200 60  0001 C CNN
@@
 HVGND
 $Comp
-L AQW216 U27
+L AQW216 CH1
 U 1 1 52E6D4A9
 P 1800 2100
-F 0 "U27" H 1800 2450 60  0000 C CNN
+F 0 "CH1" H 1800 2450 60  0000 C CNN
 F 1 "AQW216" H 1800 1745 60  0000 C CNN
 F 2 "" H 1800 2100 60  0001 C CNN
@@
 $EndComp
 $Comp
-L AQW216 U34
+L AQW216 CH15
 U 1 1 52E6DB8D
 P 4200 7500
-F 0 "U34" H 4200 7850 60  0000 C CNN
+F 0 "CH15" H 4200 7850 60  0000 C CNN
 F 1 "AQW216" H 4200 7145 60  0000 C CNN
 F 2 "" H 4200 7500 60  0001 C CNN
@@
 $EndComp
 $Comp
-L AQW216 U7
+L AQW216 CH14
 U 1 1 52E6D4DA
 P 4200 6600
-F 0 "U7" H 4200 6950 60  0000 C CNN
+F 0 "CH14" H 4200 6950 60  0000 C CNN
 F 1 "AQW216" H 4200 6245 60  0000 C CNN
 F 2 "" H 4200 6600 60  0001 C CNN
@@
 $EndComp
 $Comp
-L AQW216 U8
+L AQW216 CH12
 U 1 1 52E6D4EC
 P 4200 4800
-F 0 "U8" H 4200 5150 60  0000 C CNN
+F 0 "CH12" H 4200 5150 60  0000 C CNN
 F 1 "AQW216" H 4200 4445 60  0000 C CNN
 F 2 "" H 4200 4800 60  0001 C CNN
@@
 $EndComp
 $Comp
-L AQW216 U33
+L AQW216 CH13
 U 1 1 52E6D4FE
 P 4200 5700
-F 0 "U33" H 4200 6050 60  0000 C CNN
+F 0 "CH13" H 4200 6050 60  0000 C CNN
 F 1 "AQW216" H 4200 5345 60  0000 C CNN
 F 2 "" H 4200 5700 60  0001 C CNN
@@
 $EndComp
 $Comp
-L AQW216 U9
+L AQW216 CH10
 U 1 1 52E6DB99
 P 4200 3000
-F 0 "U9" H 4200 3350 60  0000 C CNN
+F 0 "CH10" H 4200 3350 60  0000 C CNN
 F 1 "AQW216" H 4200 2645 60  0000 C CNN
 F 2 "" H 4200 3000 60  0001 C CNN
@@
 $EndComp
 $Comp
-L AQW216 U32
+L AQW216 CH11
 U 1 1 52E6D522
 P 4200 3900
-F 0 "U32" H 4200 4250 60  0000 C CNN
+F 0 "CH11" H 4200 4250 60  0000 C CNN
 F 1 "AQW216" H 4200 3545 60  0000 C CNN
 F 2 "" H 4200 3900 60  0001 C CNN
@@
 HVGND
 $Comp
-L AQW216 U10
+L AQW216 CH8
 U 1 1 52E6DBA2
 P 4200 1200
-F 0 "U10" H 4200 1550 60  0000 C CNN
+F 0 "CH8" H 4200 1550 60  0000 C CNN
 F 1 "AQW216" H 4200 845 60  0000 C CNN
 F 2 "" H 4200 1200 60  0001 C CNN
@@
 HVGND
 $Comp
-L AQW216 U31
+L AQW216 CH9
 U 1 1 52E6D579
 P 4200 2100
-F 0 "U31" H 4200 2450 60  0000 C CNN
+F 0 "CH9" H 4200 2450 60  0000 C CNN
 F 1 "AQW216" H 4200 1745 60  0000 C CNN
 F 2 "" H 4200 2100 60  0001 C CNN
@@
 $EndComp
 $Comp
-L AQW216 U14
+L AQW216 CH18
 U 1 1 52E6D85E
 P 6600 3000
-F 0 "U14" H 6600 3350 60  0000 C CNN
+F 0 "CH18" H 6600 3350 60  0000 C CNN
 F 1 "AQW216" H 6600 2645 60  0000 C CNN
 F 2 "" H 6600 3000 60  0001 C CNN
@@
 $EndComp
 $Comp
-L AQW216 U36
+L AQW216 CH19
 U 1 1 52E6DBC0
 P 6600 3900
-F 0 "U36" H 6600 4250 60  0000 C CNN
+F 0 "CH19" H 6600 4250 60  0000 C CNN
 F 1 "AQW216" H 6600 3545 60  0000 C CNN
 F 2 "" H 6600 3900 60  0001 C CNN
@@
 HVGND
 $Comp
-L AQW216 U15
+L AQW216 CH16
 U 1 1 52E6D896
 P 6600 1200
-F 0 "U15" H 6600 1550 60  0000 C CNN
+F 0 "CH16" H 6600 1550 60  0000 C CNN
 F 1 "AQW216" H 6600 845 60  0000 C CNN
 F 2 "" H 6600 1200 60  0001 C CNN
@@
 HVGND
 $Comp
-L AQW216 U35
+L AQW216 CH17
 U 1 1 52E6DBCB
 P 6600 2100
-F 0 "U35" H 6600 2450 60  0000 C CNN
+F 0 "CH17" H 6600 2450 60  0000 C CNN
 F 1 "AQW216" H 6600 1745 60  0000 C CNN
 F 2 "" H 6600 2100 60  0001 C CNN
