File: 40-channel HV switching board-p3.sch (KiCad schematic (older format))
At the start: 34 parts, among them U10 AQW216, U31 AQW216, U32 AQW216, U33 AQW216, U34 AQW216, U6 74AC540, U7 AQW216, U8 AQW216, U9 AQW216

Commit message: Fix capcitor values on schematic, swap HV/GND on BNC jacks
Parts:
- C3: value 1uF -> 0.1uF
Changed lines of the file:
@@
-EESchema Schematic File Version 2  date 7/30/2011 2:04:39 PM
+EESchema Schematic File Version 2  date 11/18/2011 9:58:06 AM
 LIBS:power
 LIBS:device
@@
 Sheet 4 7
 Title "40-channel HV switching board"
-Date "30 jul 2011"
+Date "18 nov 2011"
 Rev "1"
 Comp "Ryan Fobel"
@@
 P 3700 1150
 F 0 "C3" H 3600 1250 50  0000 L CNN
-F 1 "1uF" H 3550 1050 50  0000 L CNN
+F 1 "0.1uF" H 3500 1050 50  0000 L CNN
 	1    3700 1150
 	0    1    1    0

Commit message: Reindex channels to start at 0 instead of 1
This makes the hardware/software channel labels consistent.
Connections:
- net labels added: HVOUT8, OUT8
- net labels removed: HVOUT16, OUT16
Changed lines of the file:
@@
-EESchema Schematic File Version 2  date 16/03/2012 12:06:03 AM
+EESchema Schematic File Version 2  date 18/01/2013 10:50:53 AM
 LIBS:power
 LIBS:device
@@
 LIBS:valves
 LIBS:wheelerlab
+LIBS:40-channel HV switching board-cache
 EELAYER 25  0
 EELAYER END
@@
 Sheet 4 7
 Title "40-channel HV switching board"
-Date "16 mar 2012"
+Date "18 jan 2013"
 Rev "1"
 Comp "Ryan Fobel"
@@
 $EndComp
 Text GLabel 3000 7100 2    60   Input ~ 0
-HVOUT16
+HVOUT15
 Text GLabel 3000 7350 2    60   Input ~ 0
 HV
@@
 $EndComp
 Text GLabel 2050 7350 0    60   Input ~ 0
-OUT16
+OUT15
 Text GLabel 2050 6150 0    60   Input ~ 0
-OUT15
+OUT14
 $Comp
 L +5V #PWR017
@@
 HV
 Text GLabel 3000 5900 2    60   Input ~ 0
-HVOUT15
+HVOUT14
 $Comp
 L R R14
@@
 $EndComp
 Text GLabel 5850 5900 2    60   Input ~ 0
-HVOUT13
+HVOUT12
 Text GLabel 5850 6150 2    60   Input ~ 0
 HV
@@
 $EndComp
 Text GLabel 4900 6150 0    60   Input ~ 0
+OUT12
+Text GLabel 4900 7350 0    60   Input ~ 0
 OUT13
-Text GLabel 4900 7350 0    60   Input ~ 0
-OUT14
 $Comp
 L +5V #PWR019
@@
 Text GLabel 5850 7350 2    60   Input ~ 0
 HV
-Text GLabel 5850 7100 2    60   Input ~ 0
-HVOUT14
+Text GLabel 5850 7100 2    60   Output ~ 0
+HVOUT13
 $Comp
 L R R78
@@
 $EndComp
 Text GLabel 9550 4000 2    60   Input ~ 0
-HVOUT11
+HVOUT10
 Text GLabel 9550 4250 2    60   Input ~ 0
 HV
@@
 $EndComp
 Text GLabel 8600 4250 0    60   Input ~ 0
+OUT10
+Text GLabel 8600 5450 0    60   Input ~ 0
 OUT11
-Text GLabel 8600 5450 0    60   Input ~ 0
-OUT12
 $Comp
 L +5V #PWR021
@@
 HV
 Text GLabel 9550 5200 2    60   Input ~ 0
-HVOUT12
+HVOUT11
 $Comp
 L R R77
@@
 $EndComp
 Text GLabel 9550 2750 2    60   Input ~ 0
-HVOUT10
+HVOUT9
 Text GLabel 9550 3000 2    60   Input ~ 0
 HV
@@
 $EndComp
 Text GLabel 8600 3000 0    60   Input ~ 0
-OUT10
+OUT9
 Text GLabel 8600 1800 0    60   Input ~ 0
-OUT9
+OUT8
 Text GLabel 1100 1700 0    60   Input ~ 0
-OUT9
+OUT8
 $Comp
 L 74AC540 U6
@@
 $EndComp
 Text GLabel 1100 2100 0    60   Input ~ 0
+OUT12
+Text GLabel 1100 2700 0    60   Input ~ 0
 OUT13
-Text GLabel 1100 2700 0    60   Input ~ 0
+Text GLabel 1100 2500 0    60   Input ~ 0
+OUT15
+Text GLabel 1100 2300 0    60   Input ~ 0
 OUT14
-Text GLabel 1100 2500 0    60   Input ~ 0
-OUT16
-Text GLabel 1100 2300 0    60   Input ~ 0
-OUT15
 Text GLabel 1100 1900 0    60   Input ~ 0
+OUT10
+Text GLabel 1100 2900 0    60   Input ~ 0
 OUT11
-Text GLabel 1100 2900 0    60   Input ~ 0
-OUT12
 Text GLabel 1100 3100 0    60   Input ~ 0
-OUT10
+OUT9
 $Comp
 L GND #PWR024
@@
 HV
 Text GLabel 9550 1550 2    60   Input ~ 0
-HVOUT9
+HVOUT8
 $Comp
 L R R17
