File: 40-channel HV switching board-p3.sch (KiCad schematic (older format))
At the start: 34 parts, among them U10 AQW216, U31 AQW216, U32 AQW216, U33 AQW216, U34 AQW216, U6 74AC540, U7 AQW216, U8 AQW216, U9 AQW216

Commit message: Reroute onto 2-layer board, remove inverters
Parts:
- removed C3: 0.1uF, symbol C
- removed R13, R18, R19, R24, R75, R80, R81, R86: 4.75k, symbol R
- removed R14, R15, R16, R17, R20, R21, R22, R23, R76, R77, R78, R79, R82, R83, R84, R85: 375, symbol R
- removed U10, U31, U32, U33, U34, U7, U8, U9: AQW216, symbol AQW216
- removed U6: 74AC540, symbol 74AC540
- added R101, R106, R107, R112, R114, R118, R120, R124, R30, R31, R37, R42, R44, R50, R51, R56, R57, R62, R92, R93: 4.75k, symbol R
- added R102, R103, R104, R105, R108, R109, R110, R111, R113, R115, R116, R117, R119, R121, R122, R123, R26, R27, R32, R33, R38, R39, R40, R41, R46, R47, R48, R49, R52, R53, R54, R55, R58, R59, R60, R61, R90, R91, R96, R97: 375, symbol R
- added U12, U13, U18, U19, U20, U21, U22, U24, U25, U26, U37, U38, U39, U40, U41, U42, U43, U44, U45, U46: AQW216, symbol AQW216
Connections:
- net labels added: HVOUT20, HVOUT21, HVOUT22, HVOUT23, HVOUT24, HVOUT25, HVOUT26, HVOUT27, HVOUT28, HVOUT29, HVOUT30, HVOUT31, HVOUT32, HVOUT33, HVOUT34, HVOUT35, HVOUT36, HVOUT37, HVOUT38, HVOUT39, OUT20, OUT21, OUT22, OUT23, OUT24, OUT25, OUT26, OUT27, OUT28, OUT29, OUT30, OUT31, OUT32, OUT33, OUT34, OUT35, OUT36, OUT37, OUT38, OUT39
- net labels removed: HVOUT10, HVOUT11, HVOUT12, HVOUT13, HVOUT14, HVOUT15, HVOUT8, HVOUT9, OUT10, OUT11, OUT12, OUT13, OUT14, OUT15, OUT8, OUT9
- wire segments 142 -> 140

Commit message: Rename PhotoMOS reference numbers to match channel number
Parts:
- renumbered U13 to CH20, U37 to CH21, U12 to CH22, U38 to CH23, U21 to CH24, U39 to CH25, U20 to CH26, U40 to CH27, U19 to CH28, U41 to CH29, U18 to CH30, U42 to CH31, U22 to CH32, U43 to CH33, U26 to CH34, U44 to CH35, U25 to CH36, U45 to CH37, U24 to CH38, U46 to CH39
Changed lines of the file:
@@
 LIBS:valves
 LIBS:wheelerlab
+LIBS:40-channel HV switching board-cache
 EELAYER 27 0
 EELAYER END
@@
 Sheet 4 4
 Title "40-channel HV switching board"
-Date "4 feb 2014"
+Date "30 apr 2014"
 Rev "1"
 Comp "Ryan Fobel"
@@
 $EndComp
 $Comp
-L AQW216 U40
+L AQW216 CH27
 U 1 1 52E6D48E
 P 1800 7500
-F 0 "U40" H 1800 7850 60  0000 C CNN
+F 0 "CH27" H 1800 7850 60  0000 C CNN
 F 1 "AQW216" H 1800 7145 60  0000 C CNN
 F 2 "" H 1800 7500 60  0001 C CNN
@@
 $EndComp
 $Comp
-L AQW216 U20
+L AQW216 CH26
 U 1 1 52E6DB60
 P 1800 6600
-F 0 "U20" H 1800 6950 60  0000 C CNN
+F 0 "CH26" H 1800 6950 60  0000 C CNN
 F 1 "AQW216" H 1800 6245 60  0000 C CNN
 F 2 "" H 1800 6600 60  0001 C CNN
@@
 $EndComp
 $Comp
-L AQW216 U21
+L AQW216 CH24
 U 1 1 52E6DB63
 P 1800 4800
-F 0 "U21" H 1800 5150 60  0000 C CNN
+F 0 "CH24" H 1800 5150 60  0000 C CNN
 F 1 "AQW216" H 1800 4445 60  0000 C CNN
 F 2 "" H 1800 4800 60  0001 C CNN
@@
 $EndComp
 $Comp
-L AQW216 U39
+L AQW216 CH25
 U 1 1 52E6DB66
 P 1800 5700
-F 0 "U39" H 1800 6050 60  0000 C CNN
+F 0 "CH25" H 1800 6050 60  0000 C CNN
 F 1 "AQW216" H 1800 5345 60  0000 C CNN
 F 2 "" H 1800 5700 60  0001 C CNN
@@
 $EndComp
 $Comp
-L AQW216 U12
+L AQW216 CH22
 U 1 1 52E6D49A
 P 1800 3000
-F 0 "U12" H 1800 3350 60  0000 C CNN
+F 0 "CH22" H 1800 3350 60  0000 C CNN
 F 1 "AQW216" H 1800 2645 60  0000 C CNN
 F 2 "" H 1800 3000 60  0001 C CNN
@@
 $EndComp
 $Comp
-L AQW216 U38
+L AQW216 CH23
 U 1 1 52E6D49D
 P 1800 3900
-F 0 "U38" H 1800 4250 60  0000 C CNN
+F 0 "CH23" H 1800 4250 60  0000 C CNN
 F 1 "AQW216" H 1800 3545 60  0000 C CNN
 F 2 "" H 1800 3900 60  0001 C CNN
@@
 HVGND
 $Comp
-L AQW216 U13
+L AQW216 CH20
 U 1 1 52E6D4A4
 P 1800 1200
-F 0 "U13" H 1800 1550 60  0000 C CNN
+F 0 "CH20" H 1800 1550 60  0000 C CNN
 F 1 "AQW216" H 1800 845 60  0000 C CNN
 F 2 "" H 1800 1200 60  0001 C CNN
@@
 HVGND
 $Comp
-L AQW216 U37
+L AQW216 CH21
 U 1 1 52E6DB78
 P 1800 2100
-F 0 "U37" H 1800 2450 60  0000 C CNN
+F 0 "CH21" H 1800 2450 60  0000 C CNN
 F 1 "AQW216" H 1800 1745 60  0000 C CNN
 F 2 "" H 1800 2100 60  0001 C CNN
@@
 $EndComp
 $Comp
-L AQW216 U44
+L AQW216 CH35
 U 1 1 52E6D4C8
 P 4200 7500
-F 0 "U44" H 4200 7850 60  0000 C CNN
+F 0 "CH35" H 4200 7850 60  0000 C CNN
 F 1 "AQW216" H 4200 7145 60  0000 C CNN
 F 2 "" H 4200 7500 60  0001 C CNN
@@
 $EndComp
 $Comp
-L AQW216 U26
+L AQW216 CH34
 U 1 1 52E6DB90
 P 4200 6600
-F 0 "U26" H 4200 6950 60  0000 C CNN
+F 0 "CH34" H 4200 6950 60  0000 C CNN
 F 1 "AQW216" H 4200 6245 60  0000 C CNN
 F 2 "" H 4200 6600 60  0001 C CNN
@@
 $EndComp
 $Comp
-L AQW216 U22
+L AQW216 CH32
 U 1 1 52E6DB93
 P 4200 4800
-F 0 "U22" H 4200 5150 60  0000 C CNN
+F 0 "CH32" H 4200 5150 60  0000 C CNN
 F 1 "AQW216" H 4200 4445 60  0000 C CNN
 F 2 "" H 4200 4800 60  0001 C CNN
@@
 $EndComp
 $Comp
-L AQW216 U43
+L AQW216 CH33
 U 1 1 52E6DB96
 P 4200 5700
-F 0 "U43" H 4200 6050 60  0000 C CNN
+F 0 "CH33" H 4200 6050 60  0000 C CNN
 F 1 "AQW216" H 4200 5345 60  0000 C CNN
 F 2 "" H 4200 5700 60  0001 C CNN
@@
 $EndComp
 $Comp
-L AQW216 U18
+L AQW216 CH30
 U 1 1 52E6D510
 P 4200 3000
-F 0 "U18" H 4200 3350 60  0000 C CNN
+F 0 "CH30" H 4200 3350 60  0000 C CNN
 F 1 "AQW216" H 4200 2645 60  0000 C CNN
 F 2 "" H 4200 3000 60  0001 C CNN
@@
 $EndComp
 $Comp
-L AQW216 U42
+L AQW216 CH31
 U 1 1 52E6DB9C
 P 4200 3900
-F 0 "U42" H 4200 4250 60  0000 C CNN
+F 0 "CH31" H 4200 4250 60  0000 C CNN
 F 1 "AQW216" H 4200 3545 60  0000 C CNN
 F 2 "" H 4200 3900 60  0001 C CNN
@@
 HVGND
 $Comp
-L AQW216 U19
+L AQW216 CH28
 U 1 1 52E6D54F
 P 4200 1200
-F 0 "U19" H 4200 1550 60  0000 C CNN
+F 0 "CH28" H 4200 1550 60  0000 C CNN
 F 1 "AQW216" H 4200 845 60  0000 C CNN
 F 2 "" H 4200 1200 60  0001 C CNN
@@
 HVGND
 $Comp
-L AQW216 U41
+L AQW216 CH29
 U 1 1 52E6DBA7
 P 4200 2100
-F 0 "U41" H 4200 2450 60  0000 C CNN
+F 0 "CH29" H 4200 2450 60  0000 C CNN
 F 1 "AQW216" H 4200 1745 60  0000 C CNN
 F 2 "" H 4200 2100 60  0001 C CNN
@@
 $EndComp
 $Comp
-L AQW216 U24
+L AQW216 CH38
 U 1 1 52E6DBBD
 P 6600 3000
-F 0 "U24" H 6600 3350 60  0000 C CNN
+F 0 "CH38" H 6600 3350 60  0000 C CNN
 F 1 "AQW216" H 6600 2645 60  0000 C CNN
 F 2 "" H 6600 3000 60  0001 C CNN
@@
 $EndComp
 $Comp
-L AQW216 U46
+L AQW216 CH39
 U 1 1 52E6D870
 P 6600 3900
-F 0 "U46" H 6600 4250 60  0000 C CNN
+F 0 "CH39" H 6600 4250 60  0000 C CNN
 F 1 "AQW216" H 6600 3545 60  0000 C CNN
 F 2 "" H 6600 3900 60  0001 C CNN
@@
 HVGND
 $Comp
-L AQW216 U25
+L AQW216 CH36
 U 1 1 52E6DBC6
 P 6600 1200
-F 0 "U25" H 6600 1550 60  0000 C CNN
+F 0 "CH36" H 6600 1550 60  0000 C CNN
 F 1 "AQW216" H 6600 845 60  0000 C CNN
 F 2 "" H 6600 1200 60  0001 C CNN
@@
 HVGND
 $Comp
-L AQW216 U45
+L AQW216 CH37
 U 1 1 52E6D8C0
 P 6600 2100
-F 0 "U45" H 6600 2450 60  0000 C CNN
+F 0 "CH37" H 6600 2450 60  0000 C CNN
 F 1 "AQW216" H 6600 1745 60  0000 C CNN
 F 2 "" H 6600 2100 60  0001 C CNN
