File: 40-channel HV switching board-p4.sch (KiCad schematic (older format))
At the start: 34 parts, among them U11 74AC540, U12 AQW216, U13 AQW216, U14 AQW216, U15 AQW216, U35 AQW216, U36 AQW216, U37 AQW216, U38 AQW216

Commit message: Fix capcitor values on schematic, swap HV/GND on BNC jacks
Parts:
- C6: value 1uF -> 0.1uF
Changed lines of the file:
@@
-EESchema Schematic File Version 2  date 7/30/2011 2:04:39 PM
+EESchema Schematic File Version 2  date 11/18/2011 9:58:06 AM
 LIBS:power
 LIBS:device
@@
 Sheet 5 7
 Title "40-channel HV switching board"
-Date "30 jul 2011"
+Date "18 nov 2011"
 Rev "1"
 Comp "Ryan Fobel"
@@
 P 3700 1150
 F 0 "C6" H 3600 1250 50  0000 L CNN
-F 1 "1uF" H 3550 1050 50  0000 L CNN
+F 1 "0.1uF" H 3500 1050 50  0000 L CNN
 	1    3700 1150
 	0    1    1    0

Commit message: Reindex channels to start at 0 instead of 1
This makes the hardware/software channel labels consistent.
Connections:
- net labels added: HVOUT16, OUT16
- net labels removed: HVOUT24, OUT24
Changed lines of the file:
@@
-EESchema Schematic File Version 2  date 16/03/2012 12:06:03 AM
+EESchema Schematic File Version 2  date 18/01/2013 10:50:53 AM
 LIBS:power
 LIBS:device
@@
 LIBS:valves
 LIBS:wheelerlab
+LIBS:40-channel HV switching board-cache
 EELAYER 25  0
 EELAYER END
@@
 Sheet 5 7
 Title "40-channel HV switching board"
-Date "16 mar 2012"
+Date "18 jan 2013"
 Rev "1"
 Comp "Ryan Fobel"
@@
 $EndComp
 Text GLabel 3000 7100 2    60   Input ~ 0
-HVOUT24
+HVOUT23
 Text GLabel 3000 7350 2    60   Input ~ 0
 HV
@@
 $EndComp
 Text GLabel 2050 7350 0    60   Input ~ 0
-OUT24
+OUT23
 Text GLabel 2050 6150 0    60   Input ~ 0
-OUT23
+OUT22
 $Comp
 L +5V #PWR028
@@
 HV
 Text GLabel 3000 5900 2    60   Input ~ 0
-HVOUT23
+HVOUT22
 $Comp
 L R R26
@@
 $EndComp
 Text GLabel 5850 5900 2    60   Input ~ 0
-HVOUT21
+HVOUT20
 Text GLabel 5850 6150 2    60   Input ~ 0
 HV
@@
 $EndComp
 Text GLabel 4900 6150 0    60   Input ~ 0
+OUT20
+Text GLabel 4900 7350 0    60   Input ~ 0
 OUT21
-Text GLabel 4900 7350 0    60   Input ~ 0
-OUT22
 $Comp
 L +5V #PWR030
@@
 HV
 Text GLabel 5850 7100 2    60   Input ~ 0
-HVOUT22
+HVOUT21
 $Comp
 L R R90
@@
 $EndComp
 Text GLabel 9550 4000 2    60   Input ~ 0
-HVOUT19
+HVOUT18
 Text GLabel 9550 4250 2    60   Input ~ 0
 HV
@@
 $EndComp
 Text GLabel 8600 4250 0    60   Input ~ 0
+OUT18
+Text GLabel 8600 5450 0    60   Input ~ 0
 OUT19
-Text GLabel 8600 5450 0    60   Input ~ 0
-OUT20
 $Comp
 L +5V #PWR032
@@
 HV
 Text GLabel 9550 5200 2    60   Input ~ 0
-HVOUT20
+HVOUT19
 $Comp
 L R R89
@@
 $EndComp
 Text GLabel 9550 2750 2    60   Input ~ 0
-HVOUT18
+HVOUT17
 Text GLabel 9550 3000 2    60   Input ~ 0
 HV
@@
 $EndComp
 Text GLabel 8600 3000 0    60   Input ~ 0
-OUT18
+OUT17
 Text GLabel 8600 1800 0    60   Input ~ 0
-OUT17
+OUT16
 Text GLabel 1100 1700 0    60   Input ~ 0
-OUT17
+OUT16
 $Comp
 L 74AC540 U11
@@
 $EndComp
 Text GLabel 1100 2100 0    60   Input ~ 0
+OUT20
+Text GLabel 1100 2700 0    60   Input ~ 0
 OUT21
-Text GLabel 1100 2700 0    60   Input ~ 0
+Text GLabel 1100 2500 0    60   Input ~ 0
+OUT23
+Text GLabel 1100 2300 0    60   Input ~ 0
 OUT22
-Text GLabel 1100 2500 0    60   Input ~ 0
-OUT24
-Text GLabel 1100 2300 0    60   Input ~ 0
-OUT23
 Text GLabel 1100 1900 0    60   Input ~ 0
+OUT18
+Text GLabel 1100 2900 0    60   Input ~ 0
 OUT19
-Text GLabel 1100 2900 0    60   Input ~ 0
-OUT20
 Text GLabel 1100 3100 0    60   Input ~ 0
-OUT18
+OUT17
 $Comp
 L GND #PWR035
@@
 HV
 Text GLabel 9550 1550 2    60   Input ~ 0
-HVOUT17
+HVOUT16
 $Comp
 L R R29
