File: 40-channel HV switching board-p5.sch (KiCad schematic (older format))
At the start: 34 parts, among them U17 74AC540, U18 AQW216, U19 AQW216, U20 AQW216, U21 AQW216, U39 AQW216, U40 AQW216, U41 AQW216, U42 AQW216

Commit message: Fix capcitor values on schematic, swap HV/GND on BNC jacks
Parts:
- C7: value 1uF -> 0.1uF
Changed lines of the file:
@@
-EESchema Schematic File Version 2  date 7/30/2011 2:04:39 PM
+EESchema Schematic File Version 2  date 11/18/2011 9:58:06 AM
 LIBS:power
 LIBS:device
@@
 Sheet 6 7
 Title "40-channel HV switching board"
-Date "30 jul 2011"
+Date "18 nov 2011"
 Rev "1"
 Comp "Ryan Fobel"
@@
 P 3700 1150
 F 0 "C7" H 3600 1250 50  0000 L CNN
-F 1 "1uF" H 3550 1050 50  0000 L CNN
+F 1 "0.1uF" H 3500 1050 50  0000 L CNN
 	1    3700 1150
 	0    1    1    0

Commit message: Reindex channels to start at 0 instead of 1
This makes the hardware/software channel labels consistent.
Connections:
- net labels added: HVOUT24, OUT24
- net labels removed: HVOUT32, OUT32
Changed lines of the file:
@@
-EESchema Schematic File Version 2  date 16/03/2012 12:06:03 AM
+EESchema Schematic File Version 2  date 18/01/2013 10:50:53 AM
 LIBS:power
 LIBS:device
@@
 LIBS:valves
 LIBS:wheelerlab
+LIBS:40-channel HV switching board-cache
 EELAYER 25  0
 EELAYER END
@@
 Sheet 6 7
 Title "40-channel HV switching board"
-Date "16 mar 2012"
+Date "18 jan 2013"
 Rev "1"
 Comp "Ryan Fobel"
@@
 	950  4150 5150 4150
 Text GLabel 1100 3100 0    60   Input ~ 0
+OUT25
+Text GLabel 1100 2300 0    60   Input ~ 0
+OUT30
+Text GLabel 1100 2700 0    60   Input ~ 0
+OUT29
+Text GLabel 1100 1900 0    60   Input ~ 0
 OUT26
-Text GLabel 1100 2300 0    60   Input ~ 0
-OUT31
-Text GLabel 1100 2700 0    60   Input ~ 0
-OUT30
-Text GLabel 1100 1900 0    60   Input ~ 0
-OUT27
 $Comp
 L R R105
@@
 $EndComp
 Text GLabel 3000 7100 2    60   Input ~ 0
-HVOUT32
+HVOUT31
 Text GLabel 3000 7350 2    60   Input ~ 0
 HV
@@
 $EndComp
 Text GLabel 2050 7350 0    60   Input ~ 0
-OUT32
+OUT31
 Text GLabel 2050 6150 0    60   Input ~ 0
-OUT31
+OUT30
 $Comp
 L +5V #PWR039
@@
 HV
 Text GLabel 3000 5900 2    60   Input ~ 0
-HVOUT31
+HVOUT30
 $Comp
 L R R38
@@
 $EndComp
 Text GLabel 5850 5900 2    60   Input ~ 0
-HVOUT29
+HVOUT28
 Text GLabel 5850 6150 2    60   Input ~ 0
 HV
@@
 $EndComp
 Text GLabel 4900 6150 0    60   Input ~ 0
+OUT28
+Text GLabel 4900 7350 0    60   Input ~ 0
 OUT29
-Text GLabel 4900 7350 0    60   Input ~ 0
-OUT30
 $Comp
 L +5V #PWR041
@@
 HV
 Text GLabel 5850 7100 2    60   Input ~ 0
-HVOUT30
+HVOUT29
 $Comp
 L R R104
@@
 $EndComp
 Text GLabel 9550 4000 2    60   Input ~ 0
-HVOUT27
+HVOUT26
 Text GLabel 9550 4250 2    60   Input ~ 0
 HV
@@
 $EndComp
 Text GLabel 8600 4250 0    60   Input ~ 0
+OUT26
+Text GLabel 8600 5450 0    60   Input ~ 0
 OUT27
-Text GLabel 8600 5450 0    60   Input ~ 0
-OUT28
 $Comp
 L +5V #PWR043
@@
 HV
 Text GLabel 9550 5200 2    60   Input ~ 0
-HVOUT28
+HVOUT27
 $Comp
 L R R103
@@
 $EndComp
 Text GLabel 9550 2750 2    60   Input ~ 0
-HVOUT26
+HVOUT25
 Text GLabel 9550 3000 2    60   Input ~ 0
 HV
@@
 $EndComp
 Text GLabel 8600 3000 0    60   Input ~ 0
-OUT26
+OUT25
 Text GLabel 8600 1800 0    60   Input ~ 0
-OUT25
+OUT24
 Text GLabel 1100 1700 0    60   Input ~ 0
-OUT25
+OUT24
 $Comp
 L 74AC540 U17
@@
 $EndComp
 Text GLabel 1100 2100 0    60   Input ~ 0
-OUT29
+OUT28
 Text GLabel 1100 2500 0    60   Input ~ 0
-OUT32
+OUT31
 Text GLabel 1100 2900 0    60   Input ~ 0
-OUT28
+OUT27
 $Comp
 L GND #PWR046
@@
 HV
 Text GLabel 9550 1550 2    60   Input ~ 0
-HVOUT25
+HVOUT24
 $Comp
 L R R41
