File: 40-channel HV switching board-p6.sch (KiCad schematic (older format))
At the start: 34 parts, among them U22 AQW216, U23 74AC540, U24 AQW216, U25 AQW216, U26 AQW216, U43 AQW216, U44 AQW216, U45 AQW216, U46 AQW216

Commit message: Fix capcitor values on schematic, swap HV/GND on BNC jacks
Parts:
- C8: value 1uF -> 0.1uF
Changed lines of the file:
@@
-EESchema Schematic File Version 2  date 7/30/2011 2:04:39 PM
+EESchema Schematic File Version 2  date 11/18/2011 9:58:06 AM
 LIBS:power
 LIBS:device
@@
 Sheet 7 7
 Title "40-channel HV switching board"
-Date "30 jul 2011"
+Date "18 nov 2011"
 Rev "1"
 Comp "Ryan Fobel"
@@
 P 3700 1150
 F 0 "C8" H 3600 1250 50  0000 L CNN
-F 1 "1uF" H 3550 1050 50  0000 L CNN
+F 1 "0.1uF" H 3500 1050 50  0000 L CNN
 	1    3700 1150
 	0    1    1    0

Commit message: Reindex channels to start at 0 instead of 1
This makes the hardware/software channel labels consistent.
Connections:
- net labels added: HVOUT32, OUT32
- net labels removed: HVOUT40, OUT40
Changed lines of the file:
@@
-EESchema Schematic File Version 2  date 16/03/2012 12:06:03 AM
+EESchema Schematic File Version 2  date 18/01/2013 10:50:53 AM
 LIBS:power
 LIBS:device
@@
 LIBS:valves
 LIBS:wheelerlab
+LIBS:40-channel HV switching board-cache
 EELAYER 25  0
 EELAYER END
@@
 Sheet 7 7
 Title "40-channel HV switching board"
-Date "16 mar 2012"
+Date "18 jan 2013"
 Rev "1"
 Comp "Ryan Fobel"
@@
 $EndComp
 Text GLabel 3000 7100 2    60   Input ~ 0
-HVOUT40
+HVOUT39
 Text GLabel 3000 7350 2    60   Input ~ 0
 HV
@@
 $EndComp
 Text GLabel 2050 7350 0    60   Input ~ 0
-OUT40
+OUT39
 Text GLabel 2050 6150 0    60   Input ~ 0
-OUT39
+OUT38
 $Comp
 L +5V #PWR050
@@
 HV
 Text GLabel 3000 5900 2    60   Input ~ 0
-HVOUT39
+HVOUT38
 $Comp
 L R R52
@@
 $EndComp
 Text GLabel 5850 5900 2    60   Input ~ 0
-HVOUT37
+HVOUT36
 Text GLabel 5850 6150 2    60   Input ~ 0
 HV
@@
 $EndComp
 Text GLabel 4900 6150 0    60   Input ~ 0
+OUT36
+Text GLabel 4900 7350 0    60   Input ~ 0
 OUT37
-Text GLabel 4900 7350 0    60   Input ~ 0
-OUT38
 $Comp
 L +5V #PWR052
@@
 HV
 Text GLabel 5850 7100 2    60   Input ~ 0
-HVOUT38
+HVOUT37
 $Comp
 L R R116
@@
 $EndComp
 Text GLabel 9550 4000 2    60   Input ~ 0
-HVOUT35
+HVOUT34
 Text GLabel 9550 4250 2    60   Input ~ 0
 HV
@@
 $EndComp
 Text GLabel 8600 4250 0    60   Input ~ 0
+OUT34
+Text GLabel 8600 5450 0    60   Input ~ 0
 OUT35
-Text GLabel 8600 5450 0    60   Input ~ 0
-OUT36
 $Comp
 L +5V #PWR054
@@
 HV
 Text GLabel 9550 5200 2    60   Input ~ 0
-HVOUT36
+HVOUT35
 $Comp
 L R R115
@@
 $EndComp
 Text GLabel 9550 2750 2    60   Input ~ 0
-HVOUT34
+HVOUT33
 Text GLabel 9550 3000 2    60   Input ~ 0
 HV
@@
 $EndComp
 Text GLabel 8600 3000 0    60   Input ~ 0
-OUT34
+OUT33
 Text GLabel 8600 1800 0    60   Input ~ 0
-OUT33
+OUT32
 Text GLabel 1100 1700 0    60   Input ~ 0
-OUT33
+OUT32
 $Comp
 L 74AC540 U23
@@
 $EndComp
 Text GLabel 1100 2100 0    60   Input ~ 0
+OUT36
+Text GLabel 1100 2700 0    60   Input ~ 0
 OUT37
-Text GLabel 1100 2700 0    60   Input ~ 0
+Text GLabel 1100 2500 0    60   Input ~ 0
+OUT39
+Text GLabel 1100 2300 0    60   Input ~ 0
 OUT38
-Text GLabel 1100 2500 0    60   Input ~ 0
-OUT40
-Text GLabel 1100 2300 0    60   Input ~ 0
-OUT39
 Text GLabel 1100 1900 0    60   Input ~ 0
+OUT34
+Text GLabel 1100 2900 0    60   Input ~ 0
 OUT35
-Text GLabel 1100 2900 0    60   Input ~ 0
-OUT36
 Text GLabel 1100 3100 0    60   Input ~ 0
-OUT34
+OUT33
 $Comp
 L GND #PWR057
@@
 HV
 Text GLabel 9550 1550 2    60   Input ~ 0
-HVOUT33
+HVOUT32
 $Comp
 L R R55
