File: 40-channel HV switching board.kicad_pcb (KiCad board)
At the start: 2 copper layers, 83.8 x 121.9 mm, 209 parts, among them IC1 ATMEG328PU, J1 CONN_4, J2 CONN_10, J3 CONN_2, J4 CONN_2, J5 CONN_40, P1 CONN_6, P2 CONN_6, SW1 DPST, U1 74HC595A, U2 74HC595A, U3 74HC595A, U4 74HC595A, U5 74HC595A, U6 7400, X1 16MHz

Commit message: Make LED current-limiting resistors 1k
Parts:
- R100, R125, R126, R127, R45: value 375 -> 1k
Changed lines of the file:
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@@
       (effects (font (size 0.762 0.762) (thickness 0.127)) (justify mirror))
     )
-    (fp_text value 375 (at 0 0) (layer B.SilkS) hide
+    (fp_text value 1k (at 0 0) (layer B.SilkS) hide
       (effects (font (size 0.762 0.762) (thickness 0.127)) (justify mirror))
     )
@@
       (effects (font (size 0.762 0.762) (thickness 0.127)))
     )
-    (fp_text value 375 (at 0 0 90) (layer F.SilkS) hide
+    (fp_text value 1k (at 0 0 90) (layer F.SilkS) hide
       (effects (font (size 0.762 0.762) (thickness 0.127)))
     )
@@
       (effects (font (size 0.762 0.762) (thickness 0.127)) (justify mirror))
     )
-    (fp_text value 375 (at 0 0) (layer B.SilkS) hide
+    (fp_text value 1k (at 0 0) (layer B.SilkS) hide
       (effects (font (size 0.762 0.762) (thickness 0.127)) (justify mirror))
     )
@@
       (effects (font (size 0.762 0.762) (thickness 0.127)) (justify mirror))
     )
-    (fp_text value 375 (at 0 0) (layer B.SilkS) hide
+    (fp_text value 1k (at 0 0) (layer B.SilkS) hide
       (effects (font (size 0.762 0.762) (thickness 0.127)) (justify mirror))
     )
@@
       (effects (font (size 0.762 0.762) (thickness 0.127)) (justify mirror))
     )
-    (fp_text value 375 (at 0 0) (layer B.SilkS) hide
+    (fp_text value 1k (at 0 0) (layer B.SilkS) hide
       (effects (font (size 0.762 0.762) (thickness 0.127)) (justify mirror))
     )

Commit message: Add decoupling capacitor to 7400 chip, label LED polarity
Parts:
- added C14: 0.1uF, SM1206, B.Cu at (77.0, 29.0)
Routing:
- net VCC: track 121.7 -> 126.4 mm, vias 6 -> 7
- net GND: track 725.3 -> 728.2 mm, vias 39 -> 40
Other:
- board text added: "1"
- board text added: "ISP"
- board text removed: "ICSP"

Commit message: Fix BOM, labels, reorganize schematic
Parts:
- JP3: value JUMPER -> ISP RESET
Connections:
- net MISO renamed D12/MISO
- net MOSI renamed D11/MOSI
- net OE renamed D8/OE
- net SCK renamed D13/SCK
- net SCL renamed A5/SCL
- net SDA renamed A4/SDA
- net SRCLR renamed D9/SRCLR
- net SS renamed D10/SS
- net S_MOSI renamed D5/S_MOSI
- net S_SCK renamed D4/S_SCK
- net S_SS renamed D3/S_SS
