File: switches_20-39.sch (KiCad schematic (older format))
At the start: 80 parts

Commit message: Update for compatibility with KiCad 4.0
Connections:
- wire segments 140 -> 259

Commit message: Update to work with KiCad 4.0
Parts:
- CH20, CH21, CH22, CH23, CH24, CH25, CH26, CH27, CH28, CH29, CH30, CH31, CH32, CH33, CH34, CH35, CH36, CH37, CH38, CH39: footprint (none) -> SMD_Packages:DIP-8_SMD
- R101, R102, R103, R104, R105, R106, R107, R108, R109, R110, R111, R112, R113, R114, R115, R116, R117, R118, R119, R120, R121, R122, R123, R124, R26, R27, R30, R31, R32, R33, R37, R38, R39, R40, R41, R42, R44, R46, R47, R48, R49, R50, R51, R52, R53, R54, R55, R56, R57, R58, R59, R60, R61, R62, R90, R91, R92, R93, R96, R97: footprint (none) -> Resistors_SMD:R_1206
Connections:
- wire segments 259 -> 260

Commit message: Use edge connector, 3.3V logic, smaller board, etc.
Parts:
- R101, R106, R107, R112, R114, R118, R120, R124, R30, R31, R37, R42, R44, R50, R51, R56, R57, R62, R92, R93: footprint Resistors_SMD:R_1206 -> Resistors_SMD:R_0805
- R102, R103, R104, R105, R108, R109, R110, R111, R113, R115, R116, R117, R119, R121, R122, R123, R26, R27, R32, R33, R38, R39, R40, R41, R46, R47, R48, R49, R52, R53, R54, R55, R58, R59, R60, R61, R90, R91, R96, R97: value 375 -> 300; footprint Resistors_SMD:R_1206 -> Resistors_SMD:R_0805
Connections:
- net labels added: +3.3V
- net labels removed: +5V
