File: switches_20-39.sch (KiCad schematic (older format))
At the start: 80 parts

Commit message: Change resistor values use standard ref prefixes
* Fix #1 and #2
Parts:
- CH20, CH21, CH22, CH23, CH24, CH25, CH26, CH27, CH28, CH29, CH30, CH31, CH32, CH33, CH34, CH35, CH36, CH37, CH38, CH39: value AQW216 -> SSR-DPST; symbol AQW216 -> SSR-DPST; Mfg_Part_No (none) -> TLP227G-2(TP1,N,F)
- R102, R103, R104, R105, R108, R109, R110, R111, R113, R115, R116, R117, R119, R121, R122, R123, R26, R27, R32, R33, R38, R39, R40, R41, R46, R47, R48, R49, R52, R53, R54, R55, R58, R59, R60, R61, R90, R91, R96, R97: value 300 -> 220

Commit message: Initial setup with kicad-helpers
Parts:
- R101, R102, R103, R104, R105, R106, R107, R108, R109, R110, R111, R112, R113, R114, R115, R116, R117, R118, R119, R120, R121, R122, R123, R124, R26, R27, R30, R31, R32, R33, R37, R38, R39, R40, R41, R42, R44, R46, R47, R48, R49, R50, R51, R52, R53, R54, R55, R56, R57, R58, R59, R60, R61, R62, R90, R91, R92, R93, R96, R97: symbol R -> Device:R
Changed lines of the file:
@@
-EESchema Schematic File Version 2
-LIBS:power
-LIBS:device
-LIBS:transistors
-LIBS:conn
-LIBS:linear
-LIBS:regul
-LIBS:74xx
-LIBS:cmos4000
-LIBS:adc-dac
-LIBS:memory
-LIBS:xilinx
-LIBS:microcontrollers
-LIBS:dsp
-LIBS:microchip
-LIBS:analog_switches
-LIBS:motorola
-LIBS:texas
-LIBS:intel
-LIBS:audio
-LIBS:interface
-LIBS:digital-audio
-LIBS:philips
-LIBS:display
-LIBS:cypress
-LIBS:siliconi
-LIBS:opto
-LIBS:atmel
-LIBS:contrib
-LIBS:valves
-LIBS:sci-bots
-LIBS:40-channel HV switching board-cache
-EELAYER 25 0
+EESchema Schematic File Version 4
+EELAYER 30 0
 EELAYER END
 $Descr USLetter 11000 8500
@@
 OUT28
 $Comp
-L R R107
+L Device:R R107
 U 1 1 52E6D48A
 P 3300 1000
@@
 $EndComp
 $Comp
-L R R103
+L Device:R R103
 U 1 1 52E6D48D
 P 1150 7050
@@
 $EndComp
 $Comp
-L R R109
+L Device:R R109
 U 1 1 52E6D48F
 P 1150 7750
@@
 $EndComp
 $Comp
-L R R48
+L Device:R R48
 U 1 1 52E6DB5F
 P 1150 6850
@@
 $EndComp
 $Comp
-L R R40
+L Device:R R40
 U 1 1 52E6D492
 P 1150 6150
@@
 $EndComp
 $Comp
-L R R41
+L Device:R R41
 U 1 1 52E6D493
 P 1150 4350
@@
 $EndComp
 $Comp
-L R R49
+L Device:R R49
 U 1 1 52E6DB64
 P 1150 5050
@@
 $EndComp
 $Comp
-L R R108
+L Device:R R108
 U 1 1 52E6DB65
 P 1150 5950
@@
 $EndComp
 $Comp
-L R R102
+L Device:R R102
 U 1 1 52E6D498
 P 1150 5250
@@
 $EndComp
 $Comp
-L R R26
+L Device:R R26
 U 1 1 52E6DB68
 P 1150 2550
@@
 $EndComp
 $Comp
-L R R32
+L Device:R R32
 U 1 1 52E6D49B
 P 1150 3250
@@
 $EndComp
 $Comp
-L R R97
+L Device:R R97
 U 1 1 52E6D49C
 P 1150 4150
@@
 $EndComp
 $Comp
-L R R91
+L Device:R R91
 U 1 1 52E6D49E
 P 1150 3450
@@
 $EndComp
 $Comp
-L R R90
+L Device:R R90
 U 1 1 52E6D49F
 P 1150 1650
@@
 HVOUT21
 $Comp
-L R R96
+L Device:R R96
 U 1 1 52E6D4A0
 P 1150 2350
@@
 OUT20
 $Comp
-L R R33
+L Device:R R33
 U 1 1 52E6D4A2
 P 1150 1450
@@
 $EndComp
 $Comp
-L R R93
+L Device:R R93
 U 1 1 52E6DB72
 P 900 1000
@@
 HVOUT20
 $Comp
-L R R27
+L Device:R R27
 U 1 1 52E6D4A5
 P 1150 750
@@
 OUT21
 $Comp
-L R R30
+L Device:R R30
 U 1 1 52E6DB77
 P 900 1900
@@
 HV
 $Comp
-L R R31
+L Device:R R31
 U 1 1 52E6D4AD
 P 900 2800
@@
 HV
 $Comp
-L R R92
+L Device:R R92
 U 1 1 52E6D4B0
 P 900 3700
@@
 HV
 $Comp
-L R R50
+L Device:R R50
 U 1 1 52E6DB82
 P 900 4600
@@
 HV
 $Comp
-L R R101
+L Device:R R101
 U 1 1 52E6DB85
 P 900 5500
@@
 HV
 $Comp
-L R R112
+L Device:R R112
 U 1 1 52E6DB88
 P 900 6400
@@
 HV
 $Comp
-L R R37
+L Device:R R37
 U 1 1 52E6DB8B
 P 900 7300
@@
 $EndComp
 $Comp
-L R R115
+L Device:R R115
 U 1 1 52E6DB8C
 P 3550 7050
@@
 $EndComp
 $Comp
-L R R121
+L Device:R R121
 U 1 1 52E6D4CE
 P 3550 7750
@@
 $EndComp
 $Comp
-L R R60
+L Device:R R60
 U 1 1 52E6D4D4
 P 3550 6850
@@
 $EndComp
 $Comp
-L R R54
+L Device:R R54
 U 1 1 52E6D4E0
 P 3550 6150
@@
 $EndComp
 $Comp
-L R R55
+L Device:R R55
 U 1 1 52E6DB92
 P 3550 4350
@@
 $EndComp
 $Comp
-L R R61
+L Device:R R61
 U 1 1 52E6DB94
 P 3550 5050
@@
 $EndComp
 $Comp
-L R R119
+L Device:R R119
 U 1 1 52E6DB95
 P 3550 5950
@@
 $EndComp
 $Comp
-L R R113
+L Device:R R113
 U 1 1 52E6DB97
 P 3550 5250
@@
 $EndComp
 $Comp
-L R R38
+L Device:R R38
 U 1 1 52E6D50A
 P 3550 2550
@@
 $EndComp
 $Comp
-L R R46
+L Device:R R46
 U 1 1 52E6DB9A
 P 3550 3250
@@
 $EndComp
 $Comp
-L R R111
+L Device:R R111
 U 1 1 52E6DB9B
 P 3550 4150
@@
 $EndComp
 $Comp
-L R R105
+L Device:R R105
 U 1 1 52E6D528
 P 3550 3450
@@
 $EndComp
 $Comp
-L R R104
+L Device:R R104
 U 1 1 52E6DB9E
 P 3550 1650
@@
 HVOUT29
 $Comp
-L R R110
+L Device:R R110
 U 1 1 52E6DB9F
 P 3550 2350
@@
 $EndComp
 $Comp
-L R R47
+L Device:R R47
 U 1 1 52E6DBA1
 P 3550 1450
@@
 HVOUT28
 $Comp
-L R R39
+L Device:R R39
 U 1 1 52E6D557
 P 3550 750
@@
 OUT29
 $Comp
-L R R42
+L Device:R R42
 U 1 1 52E6DBA6
 P 3300 1900
@@
 HV
 $Comp
-L R R44
+L Device:R R44
 U 1 1 52E6DBAB
 P 3300 2800
@@
 HV
 $Comp
-L R R106
+L Device:R R106
 U 1 1 52E6DBAE
 P 3300 3700
@@
 HV
 $Comp
-L R R62
+L Device:R R62
 U 1 1 52E6DBB1
 P 3300 4600
@@
 HV
 $Comp
-L R R114
+L Device:R R114
 U 1 1 52E6DBB4
 P 3300 5500
@@
 HV
 $Comp
-L R R124
+L Device:R R124
 U 1 1 52E6D61E
 P 3300 6400
@@
 HV
 $Comp
-L R R51
+L Device:R R51
 U 1 1 52E6DBBA
 P 3300 7300
@@
 OUT36
 $Comp
-L R R120
+L Device:R R120
 U 1 1 52E6DBBB
 P 5700 1000
@@
 $EndComp
 $Comp
-L R R52
+L Device:R R52
 U 1 1 52E6DBBC
 P 5950 2550
@@
 $EndComp
 $Comp
-L R R58
+L Device:R R58
 U 1 1 52E6DBBE
 P 5950 3250
@@
 $EndComp
 $Comp
-L R R123
+L Device:R R123
 U 1 1 52E6DBBF
 P 5950 4150
@@
 $EndComp
 $Comp
-L R R117
+L Device:R R117
 U 1 1 52E6D876
 P 5950 3450
@@
 $EndComp
 $Comp
-L R R116
+L Device:R R116
 U 1 1 52E6DBC2
 P 5950 1650
@@
 HVOUT37
 $Comp
-L R R122
+L Device:R R122
 U 1 1 52E6DBC3
 P 5950 2350
@@
 $EndComp
 $Comp
-L R R59
+L Device:R R59
 U 1 1 52E6DBC5
 P 5950 1450
@@
 HVOUT36
 $Comp
-L R R53
+L Device:R R53
 U 1 1 52E6DBC7
 P 5950 750
@@
 OUT37
 $Comp
-L R R56
+L Device:R R56
 U 1 1 52E6D8B9
 P 5700 1900
@@
 HV
 $Comp
-L R R57
+L Device:R R57
 U 1 1 52E6D8ED
 P 5700 2800
@@
 HV
 $Comp
-L R R118
+L Device:R R118
 U 1 1 52E6DBD2
 P 5700 3700

Commit message: Fix broken symbols
Parts:
- CH20, CH21, CH22, CH23, CH24, CH25, CH26, CH27, CH28, CH29, CH30, CH31, CH32, CH33, CH34, CH35, CH36, CH37, CH38, CH39: value SSR-DPST -> AQW214; symbol SSR-DPST -> sci-bots:AQW214
Connections:
- wire segments 260 -> 280
Changed lines of the file:
@@
 $EndComp
 $Comp
-L SSR-DPST CH27
+L sci-bots:AQW214 CH27
 U 1 1 52E6D48E
 P 1800 7500
 F 0 "CH27" H 1800 7850 60  0000 C CNN
-F 1 "SSR-DPST" H 1800 7145 60  0000 C CNN
+F 1 "AQW214" H 1800 7145 60  0000 C CNN
 F 2 "SMD_Packages:DIP-8_SMD" H 1800 7500 60  0001 C CNN
 F 3 "" H 1800 7500 60  0001 C CNN
@@
 $EndComp
 $Comp
-L SSR-DPST CH26
+L sci-bots:AQW214 CH26
 U 1 1 52E6DB60
 P 1800 6600
 F 0 "CH26" H 1800 6950 60  0000 C CNN
-F 1 "SSR-DPST" H 1800 6245 60  0000 C CNN
+F 1 "AQW214" H 1800 6245 60  0000 C CNN
 F 2 "SMD_Packages:DIP-8_SMD" H 1800 6600 60  0001 C CNN
 F 3 "" H 1800 6600 60  0001 C CNN
@@
 $EndComp
 $Comp
-L SSR-DPST CH24
+L sci-bots:AQW214 CH24
 U 1 1 52E6DB63
 P 1800 4800
 F 0 "CH24" H 1800 5150 60  0000 C CNN
-F 1 "SSR-DPST" H 1800 4445 60  0000 C CNN
+F 1 "AQW214" H 1800 4445 60  0000 C CNN
 F 2 "SMD_Packages:DIP-8_SMD" H 1800 4800 60  0001 C CNN
 F 3 "" H 1800 4800 60  0001 C CNN
@@
 $EndComp
 $Comp
-L SSR-DPST CH25
+L sci-bots:AQW214 CH25
 U 1 1 52E6DB66
 P 1800 5700
 F 0 "CH25" H 1800 6050 60  0000 C CNN
-F 1 "SSR-DPST" H 1800 5345 60  0000 C CNN
+F 1 "AQW214" H 1800 5345 60  0000 C CNN
 F 2 "SMD_Packages:DIP-8_SMD" H 1800 5700 60  0001 C CNN
 F 3 "" H 1800 5700 60  0001 C CNN
@@
 $EndComp
 $Comp
-L SSR-DPST CH22
+L sci-bots:AQW214 CH22
 U 1 1 52E6D49A
 P 1800 3000
 F 0 "CH22" H 1800 3350 60  0000 C CNN
-F 1 "SSR-DPST" H 1800 2645 60  0000 C CNN
+F 1 "AQW214" H 1800 2645 60  0000 C CNN
 F 2 "SMD_Packages:DIP-8_SMD" H 1800 3000 60  0001 C CNN
 F 3 "" H 1800 3000 60  0001 C CNN
@@
 $EndComp
 $Comp
-L SSR-DPST CH23
+L sci-bots:AQW214 CH23
 U 1 1 52E6D49D
 P 1800 3900
 F 0 "CH23" H 1800 4250 60  0000 C CNN
-F 1 "SSR-DPST" H 1800 3545 60  0000 C CNN
+F 1 "AQW214" H 1800 3545 60  0000 C CNN
 F 2 "SMD_Packages:DIP-8_SMD" H 1800 3900 60  0001 C CNN
 F 3 "" H 1800 3900 60  0001 C CNN
@@
 HVGND
 $Comp
-L SSR-DPST CH20
+L sci-bots:AQW214 CH20
 U 1 1 52E6D4A4
 P 1800 1200
 F 0 "CH20" H 1800 1550 60  0000 C CNN
-F 1 "SSR-DPST" H 1800 845 60  0000 C CNN
+F 1 "AQW214" H 1800 845 60  0000 C CNN
 F 2 "SMD_Packages:DIP-8_SMD" H 1800 1200 60  0001 C CNN
 F 3 "" H 1800 1200 60  0001 C CNN
@@
 HVGND
 $Comp
-L SSR-DPST CH21
+L sci-bots:AQW214 CH21
 U 1 1 52E6DB78
 P 1800 2100
 F 0 "CH21" H 1800 2450 60  0000 C CNN
-F 1 "SSR-DPST" H 1800 1745 60  0000 C CNN
+F 1 "AQW214" H 1800 1745 60  0000 C CNN
 F 2 "SMD_Packages:DIP-8_SMD" H 1800 2100 60  0001 C CNN
 F 3 "" H 1800 2100 60  0001 C CNN
@@
 $EndComp
 $Comp
-L SSR-DPST CH35
+L sci-bots:AQW214 CH35
 U 1 1 52E6D4C8
 P 4200 7500
 F 0 "CH35" H 4200 7850 60  0000 C CNN
-F 1 "SSR-DPST" H 4200 7145 60  0000 C CNN
+F 1 "AQW214" H 4200 7145 60  0000 C CNN
 F 2 "SMD_Packages:DIP-8_SMD" H 4200 7500 60  0001 C CNN
 F 3 "" H 4200 7500 60  0001 C CNN
@@
 $EndComp
 $Comp
-L SSR-DPST CH34
+L sci-bots:AQW214 CH34
 U 1 1 52E6DB90
 P 4200 6600
 F 0 "CH34" H 4200 6950 60  0000 C CNN
-F 1 "SSR-DPST" H 4200 6245 60  0000 C CNN
+F 1 "AQW214" H 4200 6245 60  0000 C CNN
 F 2 "SMD_Packages:DIP-8_SMD" H 4200 6600 60  0001 C CNN
 F 3 "" H 4200 6600 60  0001 C CNN
@@
 $EndComp
 $Comp
-L SSR-DPST CH32
+L sci-bots:AQW214 CH32
 U 1 1 52E6DB93
 P 4200 4800
 F 0 "CH32" H 4200 5150 60  0000 C CNN
-F 1 "SSR-DPST" H 4200 4445 60  0000 C CNN
+F 1 "AQW214" H 4200 4445 60  0000 C CNN
 F 2 "SMD_Packages:DIP-8_SMD" H 4200 4800 60  0001 C CNN
 F 3 "" H 4200 4800 60  0001 C CNN
@@
 $EndComp
 $Comp
-L SSR-DPST CH33
+L sci-bots:AQW214 CH33
 U 1 1 52E6DB96
 P 4200 5700
 F 0 "CH33" H 4200 6050 60  0000 C CNN
-F 1 "SSR-DPST" H 4200 5345 60  0000 C CNN
+F 1 "AQW214" H 4200 5345 60  0000 C CNN
 F 2 "SMD_Packages:DIP-8_SMD" H 4200 5700 60  0001 C CNN
 F 3 "" H 4200 5700 60  0001 C CNN
@@
 $EndComp
 $Comp
-L SSR-DPST CH30
+L sci-bots:AQW214 CH30
 U 1 1 52E6D510
 P 4200 3000
 F 0 "CH30" H 4200 3350 60  0000 C CNN
-F 1 "SSR-DPST" H 4200 2645 60  0000 C CNN
+F 1 "AQW214" H 4200 2645 60  0000 C CNN
 F 2 "SMD_Packages:DIP-8_SMD" H 4200 3000 60  0001 C CNN
 F 3 "" H 4200 3000 60  0001 C CNN
@@
 $EndComp
 $Comp
-L SSR-DPST CH31
+L sci-bots:AQW214 CH31
 U 1 1 52E6DB9C
 P 4200 3900
 F 0 "CH31" H 4200 4250 60  0000 C CNN
-F 1 "SSR-DPST" H 4200 3545 60  0000 C CNN
+F 1 "AQW214" H 4200 3545 60  0000 C CNN
 F 2 "SMD_Packages:DIP-8_SMD" H 4200 3900 60  0001 C CNN
 F 3 "" H 4200 3900 60  0001 C CNN
@@
 HVGND
 $Comp
-L SSR-DPST CH28
+L sci-bots:AQW214 CH28
 U 1 1 52E6D54F
 P 4200 1200
 F 0 "CH28" H 4200 1550 60  0000 C CNN
-F 1 "SSR-DPST" H 4200 845 60  0000 C CNN
+F 1 "AQW214" H 4200 845 60  0000 C CNN
 F 2 "SMD_Packages:DIP-8_SMD" H 4200 1200 60  0001 C CNN
 F 3 "" H 4200 1200 60  0001 C CNN
@@
 HVGND
 $Comp
-L SSR-DPST CH29
+L sci-bots:AQW214 CH29
 U 1 1 52E6DBA7
 P 4200 2100
 F 0 "CH29" H 4200 2450 60  0000 C CNN
-F 1 "SSR-DPST" H 4200 1745 60  0000 C CNN
+F 1 "AQW214" H 4200 1745 60  0000 C CNN
 F 2 "SMD_Packages:DIP-8_SMD" H 4200 2100 60  0001 C CNN
 F 3 "" H 4200 2100 60  0001 C CNN
@@
 $EndComp
 $Comp
-L SSR-DPST CH38
+L sci-bots:AQW214 CH38
 U 1 1 52E6DBBD
 P 6600 3000
 F 0 "CH38" H 6600 3350 60  0000 C CNN
-F 1 "SSR-DPST" H 6600 2645 60  0000 C CNN
+F 1 "AQW214" H 6600 2645 60  0000 C CNN
 F 2 "SMD_Packages:DIP-8_SMD" H 6600 3000 60  0001 C CNN
 F 3 "" H 6600 3000 60  0001 C CNN
@@
 $EndComp
 $Comp
-L SSR-DPST CH39
+L sci-bots:AQW214 CH39
 U 1 1 52E6D870
 P 6600 3900
 F 0 "CH39" H 6600 4250 60  0000 C CNN
-F 1 "SSR-DPST" H 6600 3545 60  0000 C CNN
+F 1 "AQW214" H 6600 3545 60  0000 C CNN
 F 2 "SMD_Packages:DIP-8_SMD" H 6600 3900 60  0001 C CNN
 F 3 "" H 6600 3900 60  0001 C CNN
@@
 HVGND
 $Comp
-L SSR-DPST CH36
+L sci-bots:AQW214 CH36
 U 1 1 52E6DBC6
 P 6600 1200
 F 0 "CH36" H 6600 1550 60  0000 C CNN
-F 1 "SSR-DPST" H 6600 845 60  0000 C CNN
+F 1 "AQW214" H 6600 845 60  0000 C CNN
 F 2 "SMD_Packages:DIP-8_SMD" H 6600 1200 60  0001 C CNN
 F 3 "" H 6600 1200 60  0001 C CNN
@@
 HVGND
 $Comp
-L SSR-DPST CH37
+L sci-bots:AQW214 CH37
 U 1 1 52E6D8C0
 P 6600 2100
 F 0 "CH37" H 6600 2450 60  0000 C CNN
-F 1 "SSR-DPST" H 6600 1745 60  0000 C CNN
+F 1 "AQW214" H 6600 1745 60  0000 C CNN
 F 2 "SMD_Packages:DIP-8_SMD" H 6600 2100 60  0001 C CNN
 F 3 "" H 6600 2100 60  0001 C CNN
@@
 GND
 Wire Wire Line
-	2200 1250 2200 1150
+	2200 1250 2200 1200
 Connection ~ 2200 1200
 Wire Wire Line
@@
 	1400 950  1400 750
 Wire Wire Line
-	2200 2150 2200 2050
+	2200 2150 2200 2100
 Connection ~ 2200 2100
 Wire Wire Line
@@
 	1400 1850 1400 1650
 Wire Wire Line
-	2200 3050 2200 2950
+	2200 3050 2200 3000
 Connection ~ 2200 3000
 Wire Wire Line
@@
 	1400 2750 1400 2550
 Wire Wire Line
-	2200 3950 2200 3850
+	2200 3950 2200 3900
 Connection ~ 2200 3900
 Wire Wire Line
@@
 	1400 3650 1400 3450
 Wire Wire Line
-	2200 4850 2200 4750
+	2200 4850 2200 4800
 Connection ~ 2200 4800
 Wire Wire Line
@@
 	1400 4550 1400 4350
 Wire Wire Line
-	2200 5750 2200 5650
+	2200 5750 2200 5700
 Connection ~ 2200 5700
 Wire Wire Line
@@
 	1400 5450 1400 5250
 Wire Wire Line
-	2200 6650 2200 6550
+	2200 6650 2200 6600
 Connection ~ 2200 6600
 Wire Wire Line
@@
 	1400 6350 1400 6150
 Wire Wire Line
-	2200 7550 2200 7450
+	2200 7550 2200 7500
 Connection ~ 2200 7500
 Wire Wire Line
@@
 	1400 7250 1400 7050
 Wire Wire Line
-	4600 1250 4600 1150
+	4600 1250 4600 1200
 Connection ~ 4600 1200
 Wire Wire Line
@@
 	3800 950  3800 750
 Wire Wire Line
-	4600 2150 4600 2050
+	4600 2150 4600 2100
 Connection ~ 4600 2100
 Wire Wire Line
@@
 	3800 1850 3800 1650
 Wire Wire Line
-	4600 3050 4600 2950
+	4600 3050 4600 3000
 Connection ~ 4600 3000
 Wire Wire Line
@@
 	3800 2750 3800 2550
 Wire Wire Line
-	4600 3950 4600 3850
+	4600 3950 4600 3900
 Connection ~ 4600 3900
 Wire Wire Line
@@
 	3800 3650 3800 3450
 Wire Wire Line
-	4600 4850 4600 4750
+	4600 4850 4600 4800
 Connection ~ 4600 4800
 Wire Wire Line
@@
 	3800 4550 3800 4350
 Wire Wire Line
-	4600 5750 4600 5650
+	4600 5750 4600 5700
 Connection ~ 4600 5700
 Wire Wire Line
@@
 	3800 5450 3800 5250
 Wire Wire Line
-	4600 6650 4600 6550
+	4600 6650 4600 6600
 Connection ~ 4600 6600
 Wire Wire Line
@@
 	3800 6350 3800 6150
 Wire Wire Line
-	4600 7550 4600 7450
+	4600 7550 4600 7500
 Connection ~ 4600 7500
 Wire Wire Line
@@
 	3800 7250 3800 7050
 Wire Wire Line
-	7000 1250 7000 1150
+	7000 1250 7000 1200
 Connection ~ 7000 1200
 Wire Wire Line
@@
 	6200 950  6200 750
 Wire Wire Line
-	7000 2150 7000 2050
+	7000 2150 7000 2100
 Connection ~ 7000 2100
 Wire Wire Line
@@
 	6200 1850 6200 1650
 Wire Wire Line
-	7000 3050 7000 2950
+	7000 3050 7000 3000
 Connection ~ 7000 3000
 Wire Wire Line
@@
 	6200 2750 6200 2550
 Wire Wire Line
-	7000 3950 7000 3850
+	7000 3950 7000 3900
 Connection ~ 7000 3900
 Wire Wire Line
@@
 Wire Wire Line
 	900  2950 900  3050
+Wire Wire Line
+	2200 1200 2200 1150
+Wire Wire Line
+	2200 2100 2200 2050
+Wire Wire Line
+	2200 3000 2200 2950
+Wire Wire Line
+	2200 3900 2200 3850
+Wire Wire Line
+	2200 4800 2200 4750
+Wire Wire Line
+	2200 5700 2200 5650
+Wire Wire Line
+	2200 6600 2200 6550
+Wire Wire Line
+	2200 7500 2200 7450
+Wire Wire Line
+	4600 1200 4600 1150
+Wire Wire Line
+	4600 2100 4600 2050
+Wire Wire Line
+	4600 3000 4600 2950
+Wire Wire Line
+	4600 3900 4600 3850
+Wire Wire Line
+	4600 4800 4600 4750
+Wire Wire Line
+	4600 5700 4600 5650
+Wire Wire Line
+	4600 6600 4600 6550
+Wire Wire Line
+	4600 7500 4600 7450
+Wire Wire Line
+	7000 1200 7000 1150
+Wire Wire Line
+	7000 2100 7000 2050
+Wire Wire Line
+	7000 3000 7000 2950
+Wire Wire Line
+	7000 3900 7000 3850
 $EndSCHEMATC

Commit message: Fix BOM
Parts:
- CH20, CH21, CH22, CH23, CH24, CH25, CH26, CH27, CH28, CH29, CH30, CH31, CH32, CH33, CH34, CH35, CH36, CH37, CH38, CH39: MPN (none) -> AQW214EAZ; Manufacturer (none) -> Panasonic; Mfg_Part_No TLP227G-2(TP1,N,F) -> (none)
- R101, R106, R107, R112, R114, R118, R120, R124, R30, R31, R37, R42, R44, R50, R51, R56, R57, R62, R92, R93: MPN (none) -> RC0805FR-074K75L; Manufacturer (none) -> Yageo
- R102, R103, R104, R105, R108, R109, R110, R111, R113, R115, R116, R117, R119, R121, R122, R123, R26, R27, R32, R33, R38, R39, R40, R41, R46, R47, R48, R49, R52, R53, R54, R55, R58, R59, R60, R61, R90, R91, R96, R97: MPN (none) -> RC0805FR-07220RL; Manufacturer (none) -> Yageo
