File: 40-channel HV switching board.sch (KiCad schematic (older format))
At the start: 44 parts, among them IC1 ATMEG328PU, J1 CONN_01X04, J2 CONN_01X10, J3 BNC, J4 BNC, J5 CONN_01X40, P1 CONN_01X06, P2 CONN_01X06, SW1 Switch_DPST, U1 74HC595A, U2 74HC595A, U3 74HC595A, U4 74HC595A, U5 74HC595A, U6 7400, X1 16MHz

Commit message: [WIP] Switch caps and LEDs to 0805 footprints
Parts:
- C1, C10, C11, C12, C13, C14, C3, C5, C6, C7, C8, C9: footprint Capacitors_SMD:C_1206 -> Capacitors_SMD:C_0805
- DS1, DS2, DS3, DS4: footprint LEDs:LED_1206 -> LEDs:LED_0805
Changed lines of the file:
@@
 F 0 "DS1" H 2900 1750 50  0000 C CNN
 F 1 "+5V" H 2900 1550 50  0000 C CNN
-F 2 "LEDs:LED_1206" H 2900 1650 60  0001 C CNN
+F 2 "LEDs:LED_0805" H 2900 1650 60  0001 C CNN
 F 3 "" H 2900 1650 60  0001 C CNN
 	1    2900 1650
@@
 F 0 "C7" H 2600 1250 50  0000 L CNN
 F 1 "0.01uF" H 2600 1050 50  0000 L CNN
-F 2 "Capacitors_SMD:C_1206" H 2550 1150 60  0001 C CNN
+F 2 "Capacitors_SMD:C_0805" H 2550 1150 60  0001 C CNN
 F 3 "" H 2550 1150 60  0001 C CNN
 	1    2550 1150
@@
 F 0 "C6" H 2250 1250 50  0000 L CNN
 F 1 "0.1uF" H 2250 1050 50  0000 L CNN
-F 2 "Capacitors_SMD:C_1206" H 2200 1150 60  0001 C CNN
+F 2 "Capacitors_SMD:C_0805" H 2200 1150 60  0001 C CNN
 F 3 "" H 2200 1150 60  0001 C CNN
 	1    2200 1150
@@
 F 0 "C3" H 1750 3700 50  0000 L CNN
 F 1 "0.1uF" H 1750 3500 50  0000 L CNN
-F 2 "Capacitors_SMD:C_1206" H 1700 3600 60  0001 C CNN
+F 2 "Capacitors_SMD:C_0805" H 1700 3600 60  0001 C CNN
 F 3 "" H 1700 3600 60  0001 C CNN
 	1    1700 3600
@@
 F 0 "C10" H 6600 1700 50  0000 L CNN
 F 1 "22pF" H 6600 1500 50  0000 L CNN
-F 2 "Capacitors_SMD:C_1206" H 6550 1600 60  0001 C CNN
+F 2 "Capacitors_SMD:C_0805" H 6550 1600 60  0001 C CNN
 F 3 "" H 6550 1600 60  0001 C CNN
 	1    6550 1600
@@
 F 0 "C11" H 6600 2300 50  0000 L CNN
 F 1 "22pF" H 6600 2100 50  0000 L CNN
-F 2 "Capacitors_SMD:C_1206" H 6550 2200 60  0001 C CNN
+F 2 "Capacitors_SMD:C_0805" H 6550 2200 60  0001 C CNN
 F 3 "" H 6550 2200 60  0001 C CNN
 	1    6550 2200
@@
 F 0 "C13" H 8500 850 50  0000 L CNN
 F 1 "0.1uF" H 8200 650 50  0000 L CNN
-F 2 "Capacitors_SMD:C_1206" H 8450 750 60  0001 C CNN
+F 2 "Capacitors_SMD:C_0805" H 8450 750 60  0001 C CNN
 F 3 "" H 8450 750 60  0001 C CNN
 	1    8450 750
@@
 F 0 "C1" H 900 6200 50  0000 L CNN
 F 1 "0.1uF" H 900 6000 50  0000 L CNN
-F 2 "Capacitors_SMD:C_1206" H 850 6100 60  0001 C CNN
+F 2 "Capacitors_SMD:C_0805" H 850 6100 60  0001 C CNN
 F 3 "" H 850 6100 60  0001 C CNN
 	1    850  6100
@@
 F 0 "C8" H 3200 6200 50  0000 L CNN
 F 1 "0.1uF" H 3200 6000 50  0000 L CNN
-F 2 "Capacitors_SMD:C_1206" H 3150 6100 60  0001 C CNN
+F 2 "Capacitors_SMD:C_0805" H 3150 6100 60  0001 C CNN
 F 3 "" H 3150 6100 60  0001 C CNN
 	1    3150 6100
@@
 F 0 "C12" H 5550 6200 50  0000 L CNN
 F 1 "0.1uF" H 5550 6000 50  0000 L CNN
-F 2 "Capacitors_SMD:C_1206" H 5500 6100 60  0001 C CNN
+F 2 "Capacitors_SMD:C_0805" H 5500 6100 60  0001 C CNN
 F 3 "" H 5500 6100 60  0001 C CNN
 	1    5500 6100
@@
 F 0 "C5" H 2000 7800 50  0000 L CNN
 F 1 "0.1uF" H 2000 7600 50  0000 L CNN
-F 2 "Capacitors_SMD:C_1206" H 1950 7700 60  0001 C CNN
+F 2 "Capacitors_SMD:C_0805" H 1950 7700 60  0001 C CNN
 F 3 "" H 1950 7700 60  0001 C CNN
 	1    1950 7700
@@
 F 0 "C9" H 4350 7800 50  0000 L CNN
 F 1 "0.1uF" H 4350 7600 50  0000 L CNN
-F 2 "Capacitors_SMD:C_1206" H 4300 7700 60  0001 C CNN
+F 2 "Capacitors_SMD:C_0805" H 4300 7700 60  0001 C CNN
 F 3 "" H 4300 7700 60  0001 C CNN
 	1    4300 7700
@@
 F 0 "DS3" H 5100 2050 50  0000 C CNN
 F 1 "PROG_MODE" H 5100 2250 50  0000 C CNN
-F 2 "LEDs:LED_1206" H 5100 2150 60  0001 C CNN
+F 2 "LEDs:LED_0805" H 5100 2150 60  0001 C CNN
 F 3 "" H 5100 2150 60  0001 C CNN
 	1    5100 2150
@@
 F 0 "DS4" H 6350 3150 50  0000 C CNN
 F 1 "RST" H 6350 2950 50  0000 C CNN
-F 2 "LEDs:LED_1206" H 6350 3050 60  0001 C CNN
+F 2 "LEDs:LED_0805" H 6350 3050 60  0001 C CNN
 F 3 "" H 6350 3050 60  0001 C CNN
 	1    6350 3050
@@
 F 0 "DS2" H 3600 1750 50  0000 C CNN
 F 1 "VCC" H 3600 1550 50  0000 C CNN
-F 2 "LEDs:LED_1206" H 3600 1650 60  0001 C CNN
+F 2 "LEDs:LED_0805" H 3600 1650 60  0001 C CNN
 F 3 "" H 3600 1650 60  0001 C CNN
 	1    3600 1650
@@
 F 0 "C14" H 4350 1900 50  0000 L CNN
 F 1 "0.1uF" H 4050 1700 50  0000 L CNN
-F 2 "Capacitors_SMD:C_1206" H 4300 1800 60  0001 C CNN
+F 2 "Capacitors_SMD:C_0805" H 4300 1800 60  0001 C CNN
 F 3 "" H 4300 1800 60  0001 C CNN
 	1    4300 1800

Commit message: Use edge connector, 3.3V logic, smaller board, etc.
Parts:
- removed C10, C11: 22pF, Capacitors_SMD:C_0805, symbol C
- removed C14: 0.1uF, Capacitors_SMD:C_0805, symbol C
- removed DS2: VCC, LEDs:LED_0805, symbol LED
- removed DS3: PROG_MODE, LEDs:LED_0805, symbol LED
- removed DS4: RST, LEDs:LED_0805, symbol LED
- removed IC1: ATMEG328PU, Housings_DIP:DIP-28_W7.62mm, symbol ATMEGA8-P
- removed J1: CONN_01X04, footprints:Molex_15-24-4441, symbol CONN_01X04
- removed J2: CONN_01X10, Connect:HE10-10C, symbol CONN_01X10
- removed J3, J4: BNC, footprints:JACK_SMA, symbol BNC
- removed J5: CONN_01X40, footprints:TFML-120-01-XXX-D-RA, symbol CONN_01X40
- removed JP2: JUMPER, Pin_Headers:Pin_Header_Straight_1x02, symbol JUMPER
- removed JP3: ISP RESET, Pin_Headers:Pin_Header_Straight_1x02, symbol JUMPER
- removed R100, R125, R126, R127: 1k, Resistors_SMD:R_1206, symbol R
- removed R99: 1Meg, Resistors_SMD:R_1206, symbol R
- removed U6: 7400, footprints:SO14E, symbol 7400
- removed X1: 16MHz, Crystals:HC-49V, symbol Crystal
- added IC1: ATMEGA328P-A, Housings_QFP:TQFP-32_7x7mm_Pitch0.8mm, symbol ATMEGA328P-A
- added P3: CONN_02X25, WheelerLab:HSEC8-125-XX-X-RA-MATE, symbol CONN_02X25
- added Y1: RESONATOR, WheelerLab:CSTCE_G15C, symbol RESONATOR
- C2, C4: footprint footprints:SM2917 -> WheelerLab:SM2917
- DS1: value +5V -> +3.3V_PWR
- JP1: footprint Pin_Headers:Pin_Header_Straight_1x02 -> Pin_Headers:Pin_Header_Straight_2x01
- R43, R45: footprint Resistors_SMD:R_1206 -> Resistors_SMD:R_0805
- SW1: footprint footprints:SW_PUSH_6mm -> WheelerLab:SW_PUSH_6mm
- U1, U2, U3, U4, U5: footprint footprints:SO16E -> WheelerLab:SO16E
Connections:
- net labels added: +3.3V, +3.3V_USB
- net labels removed: +5V, +5V_USB, VCC
- wire segments 89 -> 50
- no-connect marks 11 -> 10
Other:
- note added: "EDGE CONNECTOR"
- note added: "POWER JUMPER"
- note removed: "COMMUNICATION\nBUS"
- note removed: "FROM\nHV AMPLIFIER"
- note removed: "ISP LATCH"
- note removed: "PASS THROUGH\nTO NEXT BOARD"
- note removed: "POWER JUMPERS"

Commit message: Breakout reset pin to edge connector
Changed lines of the file:
@@
 	0    1    1    0
 $EndComp
-Text GLabel 4100 3050 0    60   Input ~ 0
-HV
-Text GLabel 4600 3050 2    60   Input ~ 0
-HVGND
 Text GLabel 4600 3350 2    60   Input ~ 0
 +3.3V
@@
 Text GLabel 9300 2850 2    60   Input ~ 0
 D4/S_SCK
+Text GLabel 4600 3050 2    60   Input ~ 0
+RST
+Text GLabel 4100 3050 0    60   Input ~ 0
+GND
 $EndSCHEMATC

Commit message: Add SPI flash memory, move edge connector to side
Parts:
- removed SW1: Switch_DPST, WheelerLab:SW_PUSH_6mm, symbol Switch_DPST
- added C10: 0.1uF, Capacitors_SMD:C_0805, symbol C
- added U6: W25Q64FV, SMD_Packages:SOIC-8-N, symbol W25Q64FV
Connections:
- net labels added: D3/595SS, D4/W25SS
- net labels removed: D3/S_SS, D4/S_SCK, D5/S_MOSI
- wire segments 50 -> 57
- no-connect marks 10 -> 11
Changed lines of the file:
@@
 Sheet 1 3
 Title "40-channel HV switching board"
-Date "2016-11-30"
+Date "2016-12-19"
 Rev "3.0"
-Comp "Ryan Fobel"
+Comp "Sci-Bots Inc."
 Comment1 ""
 Comment2 ""
@@
 HVOUT1
 Text GLabel 9300 2750 2    60   Input ~ 0
-D3/S_SS
+D3/595SS
 Text GLabel 7400 2950 0    60   Input ~ 0
 GND
-Text GLabel 1800 3100 3    60   Input ~ 0
+Text GLabel 1800 3100 2    60   Input ~ 0
 RST
 Text GLabel 9300 2300 2    60   Input ~ 0
 RST
-Text GLabel 2050 2700 2    60   Input ~ 0
+Text GLabel 1800 2800 2    60   Input ~ 0
 +3.3V
 Text GLabel 1150 2800 2    60   Input ~ 0
 +3.3V_USB
 Text GLabel 1150 2600 2    60   Input ~ 0
-GND
-Text GLabel 2650 3500 2    60   Input ~ 0
 GND
 Text GLabel 1150 3000 2    60   Input ~ 0
@@
 L R R43
 U 1 1 52E82591
-P 2050 2850
-F 0 "R43" V 2130 2850 50  0000 C CNN
-F 1 "10k" V 2050 2850 50  0000 C CNN
-F 2 "Resistors_SMD:R_0805" H 2050 2850 60  0001 C CNN
-F 3 "" H 2050 2850 60  0001 C CNN
-	1    2050 2850
+P 1800 2950
+F 0 "R43" V 1880 2950 50  0000 C CNN
+F 1 "10k" V 1800 2950 50  0000 C CNN
+F 2 "Resistors_SMD:R_0805" H 1800 2950 60  0001 C CNN
+F 3 "" H 1800 2950 60  0001 C CNN
+	1    1800 2950
 	-1   0    0    1
 $EndComp
@@
 	1    0    0    -1
 $EndComp
-NoConn ~ 5850 7650
 Text GLabel 9300 2100 2    60   Input ~ 0
 A4/SDA
@@
 Text GLabel 5500 6250 0    60   Input ~ 0
 GND
-Text GLabel 1050 5650 0    60   Input ~ 0
-D3/S_SS
 Text GLabel 900  1650 2    60   Input ~ 0
 +3.3V_USB
@@
 Text Notes 5450 3850 0    60   ~ 0
 SWITCHES
-Text GLabel 1050 5150 0    60   Input ~ 0
-D5/S_MOSI
-Text GLabel 1050 5350 0    60   Input ~ 0
-D4/S_SCK
-Text GLabel 5700 5350 0    60   Input ~ 0
-D4/S_SCK
-Text GLabel 3350 5650 0    60   Input ~ 0
-D3/S_SS
-Text GLabel 5700 5650 0    60   Input ~ 0
-D3/S_SS
-Text GLabel 2100 6950 0    60   Input ~ 0
-D4/S_SCK
-Text GLabel 4450 6950 0    60   Input ~ 0
-D4/S_SCK
-Text GLabel 2100 7250 0    60   Input ~ 0
-D3/S_SS
-Text GLabel 4450 7250 0    60   Input ~ 0
-D3/S_SS
 Text GLabel 1050 5750 0    60   Input ~ 0
 D8/OE
@@
 Text GLabel 1050 5450 0    60   Input ~ 0
 D9/SRCLR
-Text GLabel 3350 5350 0    60   Input ~ 0
-D4/S_SCK
 Text GLabel 3350 5450 0    60   Input ~ 0
 D9/SRCLR
@@
 $EndComp
 $Comp
-L Switch_DPST SW1
-U 1 1 56BA66EC
-P 2350 3300
-F 0 "SW1" H 2350 3650 50  0000 C CNN
-F 1 "Switch_DPST" H 2350 2950 50  0000 C CNN
-F 2 "WheelerLab:SW_PUSH_6mm" H 2350 3300 60  0001 C CNN
-F 3 "" H 2350 3300 60  0000 C CNN
-	1    2350 3300
-	1    0    0    -1
-$EndComp
-$Comp
 L ATMEGA328P-A IC1
 U 1 1 583628D3
@@
 Wire Wire Line
 	1150 3100 1350 3100
-Wire Wire Line
-	1650 3100 2050 3100
-Connection ~ 2050 3100
-Wire Wire Line
-	2050 3000 2050 3500
-Wire Wire Line
-	2650 3500 2650 3100
 $Comp
 L CONN_02X25 P3
@@
 Text GLabel 4600 3350 2    60   Input ~ 0
 +3.3V
-Text GLabel 9300 2950 2    60   Input ~ 0
-D5/S_MOSI
-Text GLabel 9300 2850 2    60   Input ~ 0
-D4/S_SCK
 Text GLabel 4600 3050 2    60   Input ~ 0
 RST
 Text GLabel 4100 3050 0    60   Input ~ 0
 GND
+Wire Wire Line
+	1650 3100 1800 3100
+$Comp
+L W25Q64FV U6
+U 1 1 58540758
+P 8900 4300
+F 0 "U6" H 8905 4545 60  0000 C CNN
+F 1 "W25Q64FV" H 8900 4045 60  0000 C CNN
+F 2 "SMD_Packages:SOIC-8-N" H 8890 4295 60  0001 C CNN
+F 3 "" H 8890 4295 60  0000 C CNN
+	1    8900 4300
+	1    0    0    -1
+$EndComp
+NoConn ~ 9300 2950
+$Comp
+L C C10
+U 1 1 585434C1
+P 8650 3900
+F 0 "C10" H 8550 4000 50  0000 L CNN
+F 1 "0.1uF" H 8400 3800 50  0000 L CNN
+F 2 "Capacitors_SMD:C_0805" H 8650 3900 60  0001 C CNN
+F 3 "" H 8650 3900 60  0001 C CNN
+	1    8650 3900
+	0    1    1    0
+$EndComp
+Text GLabel 8500 4450 0    60   Input ~ 0
+GND
+Text GLabel 9200 4000 2    60   Input ~ 0
++3.3V
+Text GLabel 9300 2850 2    60   Input ~ 0
+D4/W25SS
+Text GLabel 8450 4150 0    60   Input ~ 0
+D4/W25SS
+Text GLabel 8450 4250 0    60   Input ~ 0
+D11/MOSI
+Text GLabel 9200 4450 2    60   Input ~ 0
+D12/MISO
+Text GLabel 9200 4350 2    60   Input ~ 0
+D13/SCK
+Wire Wire Line
+	9200 4000 9200 4250
+Wire Wire Line
+	8600 4350 8550 4350
+Wire Wire Line
+	8550 4350 8550 4000
+Connection ~ 9200 4150
+Wire Wire Line
+	8550 4000 9200 4000
+Wire Wire Line
+	8800 3900 8800 4000
+Connection ~ 8800 4000
+Wire Wire Line
+	8500 3900 8500 4450
+Wire Wire Line
+	8500 4450 8600 4450
+Wire Wire Line
+	8450 4150 8600 4150
+Wire Wire Line
+	8450 4250 8600 4250
+Text GLabel 1050 5650 0    60   Input ~ 0
+D3/595SS
+Text GLabel 1050 5150 0    60   Input ~ 0
+D11/MOSI
+Text GLabel 1050 5350 0    60   Input ~ 0
+D13/SCK
+NoConn ~ 5850 7650
+Text GLabel 3350 5350 0    60   Input ~ 0
+D13/SCK
+Text GLabel 3350 5650 0    60   Input ~ 0
+D3/595SS
+Text GLabel 5700 5650 0    60   Input ~ 0
+D3/595SS
+Text GLabel 5700 5350 0    60   Input ~ 0
+D13/SCK
+Text GLabel 2100 7250 0    60   Input ~ 0
+D3/595SS
+Text GLabel 2100 6950 0    60   Input ~ 0
+D13/SCK
+Text GLabel 4450 7250 0    60   Input ~ 0
+D3/595SS
+Text GLabel 4450 6950 0    60   Input ~ 0
+D13/SCK
 $EndSCHEMATC

Commit message: Update BOM
Parts:
- C2, C4: Mfg_Part_No (none) -> T491D336K020AT
- C3, C6: Mfg_Part_No (none) -> CL21B104KBCNNNC
- C7: Mfg_Part_No (none) -> CL21B103KCANNNC
- DS1: Mfg_Part_No (none) -> 150080BS75000
- IC1: Mfg_Part_No (none) -> ATMEGA328P-AU
- R43: Mfg_Part_No (none) -> RC0805FR-0710KL
- R45: Mfg_Part_No (none) -> RC0805FR-071KL
- U1, U2, U3, U4, U5: Mfg_Part_No (none) -> MM74HC595MX
- U6: Mfg_Part_No (none) -> W25Q64FVSSIG TR
Changed lines of the file:
@@
 F 2 "LEDs:LED_0805" H 2800 1400 60  0001 C CNN
 F 3 "" H 2800 1400 60  0001 C CNN
+F 4 "150080BS75000" H 2800 1400 60  0001 C CNN "Mfg_Part_No"
 	1    2800 1400
 	0    1    1    0
@@
 F 2 "Resistors_SMD:R_0805" H 2800 1050 60  0001 C CNN
 F 3 "" H 2800 1050 60  0001 C CNN
+F 4 "RC0805FR-071KL" V 2800 1050 60  0001 C CNN "Mfg_Part_No"
 	1    2800 1050
 	1    0    0    -1
@@
 F 2 "Capacitors_SMD:C_0805" H 1950 1100 60  0001 C CNN
 F 3 "" H 1950 1100 60  0001 C CNN
+F 4 "CL21B103KCANNNC" H 1950 1100 60  0001 C CNN "Mfg_Part_No"
 	1    1950 1100
 	1    0    0    -1
@@
 F 2 "WheelerLab:SM2917" H 1250 1100 60  0001 C CNN
 F 3 "" H 1250 1100 60  0001 C CNN
+F 4 "T491D336K020AT" H 1250 1100 60  0001 C CNN "Mfg_Part_No"
 	1    1250 1100
 	1    0    0    -1
@@
 F 2 "WheelerLab:SM2917" H 900 1100 60  0001 C CNN
 F 3 "" H 900 1100 60  0001 C CNN
+F 4 "T491D336K020AT" H 900 1100 60  0001 C CNN "Mfg_Part_No"
 	1    900  1100
 	1    0    0    -1
@@
 F 2 "Capacitors_SMD:C_0805" H 1600 1100 60  0001 C CNN
 F 3 "" H 1600 1100 60  0001 C CNN
+F 4 "CL21B104KBCNNNC" H 1600 1100 60  0001 C CNN "Mfg_Part_No"
 	1    1600 1100
 	1    0    0    -1
@@
 F 2 "Resistors_SMD:R_0805" H 1800 2950 60  0001 C CNN
 F 3 "" H 1800 2950 60  0001 C CNN
+F 4 "RC0805FR-0710KL" V 1800 2950 60  0001 C CNN "Mfg_Part_No"
 	1    1800 2950
 	-1   0    0    1
@@
 F 2 "Capacitors_SMD:C_0805" H 1500 3100 60  0001 C CNN
 F 3 "" H 1500 3100 60  0001 C CNN
+F 4 "CL21B104KBCNNNC" V 1500 3100 60  0001 C CNN "Mfg_Part_No"
 	1    1500 3100
 	0    -1   -1   0
@@
 F 2 "WheelerLab:SO16E" H 1750 5600 60  0001 C CNN
 F 3 "~" H 1750 5600 60  0000 C CNN
+F 4 "MM74HC595MX" H 1750 5600 60  0001 C CNN "Mfg_Part_No"
 	1    1750 5600
 	1    0    0    -1
@@
 F 2 "WheelerLab:SO16E" H 4050 5600 60  0001 C CNN
 F 3 "~" H 4050 5600 60  0000 C CNN
+F 4 "MM74HC595MX" H 4050 5600 60  0001 C CNN "Mfg_Part_No"
 	1    4050 5600
 	1    0    0    -1
@@
 F 2 "WheelerLab:SO16E" H 6400 5600 60  0001 C CNN
 F 3 "~" H 6400 5600 60  0000 C CNN
+F 4 "MM74HC595MX" H 6400 5600 60  0001 C CNN "Mfg_Part_No"
 	1    6400 5600
 	1    0    0    -1
@@
 F 2 "WheelerLab:SO16E" H 2800 7200 60  0001 C CNN
 F 3 "~" H 2800 7200 60  0000 C CNN
+F 4 "MM74HC595MX" H 2800 7200 60  0001 C CNN "Mfg_Part_No"
 	1    2800 7200
 	1    0    0    -1
@@
 F 2 "WheelerLab:SO16E" H 5150 7200 60  0001 C CNN
 F 3 "~" H 5150 7200 60  0000 C CNN
+F 4 "MM74HC595MX" H 5150 7200 60  0001 C CNN "Mfg_Part_No"
 	1    5150 7200
 	1    0    0    -1
@@
 F 2 "Housings_QFP:TQFP-32_7x7mm_Pitch0.8mm" H 8300 500 50  0000 C CIN
 F 3 "" H 8300 1950 50  0000 C CNN
+F 4 "ATMEGA328P-AU" H 8300 1950 60  0001 C CNN "Mfg_Part_No"
 	1    8300 1950
 	1    0    0    -1
@@
 F 2 "SMD_Packages:SOIC-8-N" H 8890 4295 60  0001 C CNN
 F 3 "" H 8890 4295 60  0000 C CNN
+F 4 "W25Q64FVSSIG TR" H 8900 4300 60  0001 C CNN "Mfg_Part_No"
 	1    8900 4300
 	1    0    0    -1
