File: 40-channel HV switching board.sch (KiCad schematic (older format))
At the start: 27 parts, among them IC1 ATMEGA328P-A, P1 CONN_01X06, P2 CONN_01X06, P3 CONN_02X25, U1 74HC595A, U2 74HC595A, U3 74HC595A, U4 74HC595A, U5 74HC595A, U6 W25Q64FV, Y1 RESONATOR

Commit message: [WIP] Improved layout for EMC
* ground mounting holes
* Add 3.3V and GND power planes
* use solder jumper instead of header pins
* replace edge connector
* extend length of board
* move programming header so that it doesn't extend past the edge of the board
Parts:
- removed P3: CONN_02X25, WheelerLab:HSEC8-125-XX-X-RA-MATE, symbol CONN_02X25
- added J1: TFM-125-02-X-DH, WheelerLab:TFM-125-02-X-DH, symbol TFM-125-02-X-DH
- added P3, P4, P5, P6: CONN_01X01, Connect:1pin, symbol CONN_01X01
- JP1: footprint Pin_Headers:Pin_Header_Straight_2x01 -> Resistors_SMD:R_0805
Connections:
- wire segments 57 -> 58
Other:
- note added: "MOUNTING HOLES"
Changed lines of the file:
@@
 LIBS:valves
 LIBS:wheelerlab
+LIBS:40-channel HV switching board-cache
 EELAYER 25 0
 EELAYER END
@@
 	1    0    0    -1
 $EndComp
-Text GLabel 4600 2950 2    60   Input ~ 0
+Text GLabel 5200 2950 2    60   Input ~ 0
 HVGND
-Text GLabel 4600 2650 2    60   Input ~ 0
+Text GLabel 5200 2650 2    60   Input ~ 0
 HVOUT35
-Text GLabel 4100 2750 0    60   Input ~ 0
+Text GLabel 4400 2750 0    60   Input ~ 0
 HVOUT36
-Text GLabel 4100 2850 0    60   Input ~ 0
+Text GLabel 4400 2850 0    60   Input ~ 0
 HVOUT38
-Text GLabel 4600 2750 2    60   Input ~ 0
+Text GLabel 5200 2750 2    60   Input ~ 0
 HVOUT37
-Text GLabel 4100 950  0    60   Input ~ 0
+Text GLabel 4400 950  0    60   Input ~ 0
 HVOUT0
-Text GLabel 4600 2850 2    60   Input ~ 0
+Text GLabel 5200 2850 2    60   Input ~ 0
 HVOUT39
-Text GLabel 4100 2650 0    60   Input ~ 0
+Text GLabel 4400 2650 0    60   Input ~ 0
 HVOUT34
-Text GLabel 4600 2550 2    60   Input ~ 0
+Text GLabel 5200 2550 2    60   Input ~ 0
 HVOUT33
-Text GLabel 4600 1750 2    60   Input ~ 0
+Text GLabel 5200 1750 2    60   Input ~ 0
 HVOUT17
-Text GLabel 4100 1850 0    60   Input ~ 0
+Text GLabel 4400 1850 0    60   Input ~ 0
 HVOUT18
-Text GLabel 4100 1950 0    60   Input ~ 0
+Text GLabel 4400 1950 0    60   Input ~ 0
 HVOUT20
-Text GLabel 4600 1850 2    60   Input ~ 0
+Text GLabel 5200 1850 2    60   Input ~ 0
 HVOUT19
-Text GLabel 4600 2050 2    60   Input ~ 0
+Text GLabel 5200 2050 2    60   Input ~ 0
 HVOUT23
-Text GLabel 4100 2150 0    60   Input ~ 0
+Text GLabel 4400 2150 0    60   Input ~ 0
 HVOUT24
-Text GLabel 4100 2050 0    60   Input ~ 0
+Text GLabel 4400 2050 0    60   Input ~ 0
 HVOUT22
-Text GLabel 4600 1950 2    60   Input ~ 0
+Text GLabel 5200 1950 2    60   Input ~ 0
 HVOUT21
-Text GLabel 4600 2350 2    60   Input ~ 0
+Text GLabel 5200 2350 2    60   Input ~ 0
 HVOUT29
-Text GLabel 4100 2450 0    60   Input ~ 0
+Text GLabel 4400 2450 0    60   Input ~ 0
 HVOUT30
-Text GLabel 4100 2550 0    60   Input ~ 0
+Text GLabel 4400 2550 0    60   Input ~ 0
 HVOUT32
-Text GLabel 4600 2450 2    60   Input ~ 0
+Text GLabel 5200 2450 2    60   Input ~ 0
 HVOUT31
-Text GLabel 4600 2250 2    60   Input ~ 0
+Text GLabel 5200 2250 2    60   Input ~ 0
 HVOUT27
-Text GLabel 4100 2350 0    60   Input ~ 0
+Text GLabel 4400 2350 0    60   Input ~ 0
 HVOUT28
-Text GLabel 4100 2250 0    60   Input ~ 0
+Text GLabel 4400 2250 0    60   Input ~ 0
 HVOUT26
-Text GLabel 4600 2150 2    60   Input ~ 0
+Text GLabel 5200 2150 2    60   Input ~ 0
 HVOUT25
-Text GLabel 4600 1350 2    60   Input ~ 0
+Text GLabel 5200 1350 2    60   Input ~ 0
 HVOUT9
-Text GLabel 4100 1450 0    60   Input ~ 0
+Text GLabel 4400 1450 0    60   Input ~ 0
 HVOUT10
-Text GLabel 4100 1550 0    60   Input ~ 0
+Text GLabel 4400 1550 0    60   Input ~ 0
 HVOUT12
-Text GLabel 4600 1450 2    60   Input ~ 0
+Text GLabel 5200 1450 2    60   Input ~ 0
 HVOUT11
-Text GLabel 4600 1650 2    60   Input ~ 0
+Text GLabel 5200 1650 2    60   Input ~ 0
 HVOUT15
-Text GLabel 4100 1750 0    60   Input ~ 0
+Text GLabel 4400 1750 0    60   Input ~ 0
 HVOUT16
-Text GLabel 4100 1650 0    60   Input ~ 0
+Text GLabel 4400 1650 0    60   Input ~ 0
 HVOUT14
-Text GLabel 4600 1550 2    60   Input ~ 0
+Text GLabel 5200 1550 2    60   Input ~ 0
 HVOUT13
-Text GLabel 4600 1150 2    60   Input ~ 0
+Text GLabel 5200 1150 2    60   Input ~ 0
 HVOUT5
-Text GLabel 4100 1250 0    60   Input ~ 0
+Text GLabel 4400 1250 0    60   Input ~ 0
 HVOUT6
-Text GLabel 4100 1350 0    60   Input ~ 0
+Text GLabel 4400 1350 0    60   Input ~ 0
 HVOUT8
-Text GLabel 4600 1250 2    60   Input ~ 0
+Text GLabel 5200 1250 2    60   Input ~ 0
 HVOUT7
-Text GLabel 4600 1050 2    60   Input ~ 0
+Text GLabel 5200 1050 2    60   Input ~ 0
 HVOUT3
-Text GLabel 4100 1150 0    60   Input ~ 0
+Text GLabel 4400 1150 0    60   Input ~ 0
 HVOUT4
-Text GLabel 4100 1050 0    60   Input ~ 0
+Text GLabel 4400 1050 0    60   Input ~ 0
 HVOUT2
-Text GLabel 4100 2950 0    60   Input ~ 0
+Text GLabel 4400 2950 0    60   Input ~ 0
 HV
-Text GLabel 4600 950  2    60   Input ~ 0
+Text GLabel 5200 950  2    60   Input ~ 0
 HVOUT1
 Text GLabel 9300 2750 2    60   Input ~ 0
@@
 Text GLabel 9300 2100 2    60   Input ~ 0
 A4/SDA
-Text GLabel 4600 3250 2    60   Input ~ 0
+Text GLabel 5200 3250 2    60   Input ~ 0
 +3.3V
 $Comp
@@
 Text GLabel 2100 7050 0    60   Input ~ 0
 D9/SRCLR
-Text GLabel 4100 3350 0    60   Input ~ 0
+Text GLabel 4400 3350 0    60   Input ~ 0
 A4/SDA
-Text GLabel 4600 3150 2    60   Input ~ 0
+Text GLabel 5200 3150 2    60   Input ~ 0
 A5/SCL
 Text GLabel 1150 4250 2    60   Input ~ 0
@@
 Wire Wire Line
 	1150 3100 1350 3100
-$Comp
-L CONN_02X25 P3
-U 1 1 58374A5A
-P 4350 2150
-F 0 "P3" H 4350 3450 50  0000 C CNN
-F 1 "CONN_02X25" V 4350 2150 50  0000 C CNN
-F 2 "WheelerLab:HSEC8-125-XX-X-RA-MATE" H 4350 1400 50  0001 C CNN
-F 3 "" H 4350 1400 50  0000 C CNN
-	1    4350 2150
-	1    0    0    -1
-$EndComp
 Wire Wire Line
 	900  1300 2350 1300
-Text GLabel 4100 3250 0    60   Input ~ 0
-GND
-Text GLabel 4100 3150 0    60   Input ~ 0
+Text GLabel 4400 3250 0    60   Input ~ 0
+GND
+Text GLabel 4400 3150 0    60   Input ~ 0
 GND
 Text Notes 3700 800  0    60   ~ 0
@@
 F 0 "JP1" H 900 2100 50  0000 C CNN
 F 1 "JUMPER" H 900 1870 50  0000 C CNN
-F 2 "Pin_Headers:Pin_Header_Straight_2x01" H 900 1950 50  0001 C CNN
+F 2 "Resistors_SMD:R_0805" H 900 1950 50  0001 C CNN
 F 3 "" H 900 1950 50  0000 C CNN
 	1    900  1950
 	0    1    1    0
 $EndComp
-Text GLabel 4600 3350 2    60   Input ~ 0
-+3.3V
-Text GLabel 4600 3050 2    60   Input ~ 0
+Text GLabel 5200 3350 2    60   Input ~ 0
++3.3V
+Text GLabel 5200 3050 2    60   Input ~ 0
 RST
-Text GLabel 4100 3050 0    60   Input ~ 0
+Text GLabel 4400 3050 0    60   Input ~ 0
 GND
 Wire Wire Line
@@
 Text GLabel 4450 6950 0    60   Input ~ 0
 D13/SCK
+$Comp
+L TFM-125-02-X-DH J1
+U 1 1 58B6BC14
+P 4400 950
+F 0 "J1" H 4600 1100 45  0000 L BNN
+F 1 "TFM-125-02-X-DH" H 4600 -1650 45  0000 L BNN
+F 2 "WheelerLab:TFM-125-02-X-DH" H 4430 1100 20  0001 C CNN
+F 3 "" H 4400 950 60  0000 C CNN
+	1    4400 950
+	1    0    0    -1
+$EndComp
+$Comp
+L CONN_01X01 P3
+U 1 1 58B6C9D8
+P 3100 2600
+F 0 "P3" H 3100 2700 50  0000 C CNN
+F 1 "CONN_01X01" H 3400 2600 50  0000 C CNN
+F 2 "Connect:1pin" H 3100 2600 50  0001 C CNN
+F 3 "" H 3100 2600 50  0000 C CNN
+	1    3100 2600
+	1    0    0    -1
+$EndComp
+$Comp
+L CONN_01X01 P4
+U 1 1 58B6CAF5
+P 3100 2800
+F 0 "P4" H 3100 2900 50  0000 C CNN
+F 1 "CONN_01X01" H 3400 2800 50  0000 C CNN
+F 2 "Connect:1pin" H 3100 2800 50  0001 C CNN
+F 3 "" H 3100 2800 50  0000 C CNN
+	1    3100 2800
+	1    0    0    -1
+$EndComp
+$Comp
+L CONN_01X01 P5
+U 1 1 58B6CB3C
+P 3100 3000
+F 0 "P5" H 3100 3100 50  0000 C CNN
+F 1 "CONN_01X01" H 3400 3000 50  0000 C CNN
+F 2 "Connect:1pin" H 3100 3000 50  0001 C CNN
+F 3 "" H 3100 3000 50  0000 C CNN
+	1    3100 3000
+	1    0    0    -1
+$EndComp
+$Comp
+L CONN_01X01 P6
+U 1 1 58B6CB42
+P 3100 3200
+F 0 "P6" H 3100 3300 50  0000 C CNN
+F 1 "CONN_01X01" H 3400 3200 50  0000 C CNN
+F 2 "Connect:1pin" H 3100 3200 50  0001 C CNN
+F 3 "" H 3100 3200 50  0000 C CNN
+	1    3100 3200
+	1    0    0    -1
+$EndComp
+Wire Wire Line
+	2900 2600 2900 3200
+Connection ~ 2900 2800
+Connection ~ 2900 3000
+Text GLabel 2900 2600 0    60   Input ~ 0
+GND
+Text Notes 2650 2450 0    60   ~ 0
+MOUNTING HOLES
 $EndSCHEMATC

Commit message: Lots of fixes to prepare for EMC testing
* read output of shift registers
* fix flash chip connection
* replace jumpers with 0805 pads
* reduce length to 92mm
* filter i2c lines
* protect i2c lines
* add ferrites to SPI lines
* add chasis ground ring
Parts:
- added C11, C16: 0.1uF, Capacitors_SMD:C_0805, symbol C
- added C14, C15: C, Capacitors_SMD:C_0805, symbol C
- added FB1, FB2, FB3, FB4, FB5: FERRITE, Resistors_SMD:R_0805, symbol FERRITE
- added R100, R125, R126, R99: R, Resistors_SMD:R_0805, symbol R
- C13: Mfg_Part_No (none) -> CL21B104KBCNNNC
Connections:
- net labels added: CHASIS_GND
- wire segments 58 -> 74
- no-connect marks 11 -> 10

Commit message: Fix BOM, version number on schematics
Parts:
- C14, C15: Mfg_Part_No CL21B104KBCNNNC -> (none)
- FB1, FB2, FB3, FB4: Mfg_Part_No (none) -> RC0805JR-070RL
- FB5: Mfg_Part_No (none) -> 742792040
- J1: Mfg_Part_No (none) -> TFM-125-02-L-DH
- R100, R125, R126, R99: value R -> 0R; Mfg_Part_No (none) -> RC0805JR-070RL
Changed lines of the file:
@@
 Sheet 1 3
 Title "40-channel HV switching board"
-Date "2017-03-07"
+Date "2017-04-05"
 Rev "3.1"
 Comp "Sci-Bots Inc."
@@
 F 2 "WheelerLab:TFM-125-02-X-DH" H 4430 1100 20  0001 C CNN
 F 3 "" H 4400 950 60  0000 C CNN
+F 4 "TFM-125-02-L-DH" H 4400 950 60  0001 C CNN "Mfg_Part_No"
 	1    4400 950
 	1    0    0    -1
@@
 F 2 "Resistors_SMD:R_0805" H 9450 1050 60  0001 C CNN
 F 3 "" H 9450 1050 60  0000 C CNN
+F 4 "RC0805JR-070RL" H 9450 1150 60  0001 C CNN "Mfg_Part_No"
 	1    9450 1150
 	1    0    0    -1
@@
 F 2 "Resistors_SMD:R_0805" H 6000 7550 60  0001 C CNN
 F 3 "" H 6000 7550 60  0000 C CNN
+F 4 "RC0805JR-070RL" H 6000 7650 60  0001 C CNN "Mfg_Part_No"
 	1    6000 7650
 	1    0    0    -1
@@
 F 2 "Resistors_SMD:R_0805" H 9450 1250 60  0001 C CNN
 F 3 "" H 9450 1250 60  0000 C CNN
+F 4 "RC0805JR-070RL" H 9450 1350 60  0001 C CNN "Mfg_Part_No"
 	1    9450 1350
 	1    0    0    -1
@@
 F 2 "Capacitors_SMD:C_0805" H 9650 2350 60  0001 C CNN
 F 3 "" H 9650 2350 60  0001 C CNN
-F 4 "CL21B104KBCNNNC" H 9650 2350 60  0001 C CNN "Mfg_Part_No"
 	1    9650 2350
 	-1   0    0    1
@@
 F 2 "Capacitors_SMD:C_0805" H 9650 1950 60  0001 C CNN
 F 3 "" H 9650 1950 60  0001 C CNN
-F 4 "CL21B104KBCNNNC" H 9650 1950 60  0001 C CNN "Mfg_Part_No"
 	1    9650 1950
 	1    0    0    -1
@@
 P 9450 2100
 F 0 "R99" V 9400 2250 50  0000 C CNN
-F 1 "R" V 9450 2100 50  0000 C CNN
+F 1 "0R" V 9450 2100 50  0000 C CNN
 F 2 "Resistors_SMD:R_0805" H 9450 2100 60  0001 C CNN
 F 3 "" H 9450 2100 60  0001 C CNN
+F 4 "RC0805JR-070RL" H 9450 2100 60  0001 C CNN "Mfg_Part_No"
 	1    9450 2100
 	0    1    1    0
@@
 P 9450 2200
 F 0 "R100" V 9400 2350 50  0000 C CNN
-F 1 "R" V 9450 2200 50  0000 C CNN
+F 1 "0R" V 9450 2200 50  0000 C CNN
 F 2 "Resistors_SMD:R_0805" H 9450 2200 60  0001 C CNN
 F 3 "" H 9450 2200 60  0001 C CNN
+F 4 "RC0805JR-070RL" H 9450 2200 60  0001 C CNN "Mfg_Part_No"
 	1    9450 2200
 	0    1    1    0
@@
 P 9850 2100
 F 0 "R125" V 9800 2250 50  0000 C CNN
-F 1 "R" V 9850 2100 50  0000 C CNN
+F 1 "0R" V 9850 2100 50  0000 C CNN
 F 2 "Resistors_SMD:R_0805" H 9850 2100 60  0001 C CNN
 F 3 "" H 9850 2100 60  0001 C CNN
+F 4 "RC0805JR-070RL" H 9850 2100 60  0001 C CNN "Mfg_Part_No"
 	1    9850 2100
 	0    1    1    0
@@
 P 9850 2200
 F 0 "R126" V 9800 2350 50  0000 C CNN
-F 1 "R" V 9850 2200 50  0000 C CNN
+F 1 "0R" V 9850 2200 50  0000 C CNN
 F 2 "Resistors_SMD:R_0805" H 9850 2200 60  0001 C CNN
 F 3 "" H 9850 2200 60  0001 C CNN
+F 4 "RC0805JR-070RL" H 9850 2200 60  0001 C CNN "Mfg_Part_No"
 	1    9850 2200
 	0    1    1    0
@@
 F 2 "Resistors_SMD:R_0805" H 8450 4150 60  0001 C CNN
 F 3 "" H 8450 4150 60  0000 C CNN
+F 4 "RC0805JR-070RL" H 8450 4250 60  0001 C CNN "Mfg_Part_No"
 	1    8450 4250
 	-1   0    0    1
@@
 F 2 "Resistors_SMD:R_0805" H 3400 3350 60  0001 C CNN
 F 3 "" H 3400 3350 60  0000 C CNN
+F 4 "742792040" H 3400 3450 60  0001 C CNN "Mfg_Part_No"
 	1    3400 3450
 	1    0    0    -1

Commit message: Update part numbers for i2c filters
Parts:
- C14, C15: value C -> 150pF; Mfg_Part_No (none) -> CL21C151JBANNNC
- R100, R99: value 0R -> 51; Mfg_Part_No RC0805JR-070RL -> RC0805FR-0751RL
- R125, R126: value 0R -> 150; Mfg_Part_No RC0805JR-070RL -> RC0805FR-07150RL
Changed lines of the file:
@@
 P 9650 2350
 F 0 "C15" H 9550 2450 50  0000 L CNN
-F 1 "C" H 9500 2350 50  0000 L CNN
+F 1 "150pF" H 9300 2350 50  0000 L CNN
 F 2 "Capacitors_SMD:C_0805" H 9650 2350 60  0001 C CNN
 F 3 "" H 9650 2350 60  0001 C CNN
+F 4 "CL21C151JBANNNC" H 9650 2350 60  0001 C CNN "Mfg_Part_No"
 	1    9650 2350
 	-1   0    0    1
@@
 P 9650 1950
 F 0 "C14" H 9500 2050 50  0000 L CNN
-F 1 "C" H 9450 1950 50  0000 L CNN
+F 1 "150pF" H 9350 1950 50  0000 L CNN
 F 2 "Capacitors_SMD:C_0805" H 9650 1950 60  0001 C CNN
 F 3 "" H 9650 1950 60  0001 C CNN
+F 4 "CL21C151JBANNNC" H 9650 1950 60  0001 C CNN "Mfg_Part_No"
 	1    9650 1950
 	1    0    0    -1
@@
 P 9450 2100
 F 0 "R99" V 9400 2250 50  0000 C CNN
-F 1 "0R" V 9450 2100 50  0000 C CNN
+F 1 "51" V 9450 2100 50  0000 C CNN
 F 2 "Resistors_SMD:R_0805" H 9450 2100 60  0001 C CNN
 F 3 "" H 9450 2100 60  0001 C CNN
-F 4 "RC0805JR-070RL" H 9450 2100 60  0001 C CNN "Mfg_Part_No"
+F 4 "RC0805FR-0751RL" H 9450 2100 60  0001 C CNN "Mfg_Part_No"
 	1    9450 2100
 	0    1    1    0
@@
 P 9450 2200
 F 0 "R100" V 9400 2350 50  0000 C CNN
-F 1 "0R" V 9450 2200 50  0000 C CNN
+F 1 "51" V 9450 2200 50  0000 C CNN
 F 2 "Resistors_SMD:R_0805" H 9450 2200 60  0001 C CNN
 F 3 "" H 9450 2200 60  0001 C CNN
-F 4 "RC0805JR-070RL" H 9450 2200 60  0001 C CNN "Mfg_Part_No"
+F 4 "RC0805FR-0751RL" H 9450 2200 60  0001 C CNN "Mfg_Part_No"
 	1    9450 2200
 	0    1    1    0
@@
 P 9850 2100
 F 0 "R125" V 9800 2250 50  0000 C CNN
-F 1 "0R" V 9850 2100 50  0000 C CNN
+F 1 "150" V 9850 2100 50  0000 C CNN
 F 2 "Resistors_SMD:R_0805" H 9850 2100 60  0001 C CNN
 F 3 "" H 9850 2100 60  0001 C CNN
-F 4 "RC0805JR-070RL" H 9850 2100 60  0001 C CNN "Mfg_Part_No"
+F 4 "RC0805FR-07150RL" H 9850 2100 60  0001 C CNN "Mfg_Part_No"
 	1    9850 2100
 	0    1    1    0
@@
 P 9850 2200
 F 0 "R126" V 9800 2350 50  0000 C CNN
-F 1 "0R" V 9850 2200 50  0000 C CNN
+F 1 "150" V 9850 2200 50  0000 C CNN
 F 2 "Resistors_SMD:R_0805" H 9850 2200 60  0001 C CNN
 F 3 "" H 9850 2200 60  0001 C CNN
-F 4 "RC0805JR-070RL" H 9850 2200 60  0001 C CNN "Mfg_Part_No"
+F 4 "RC0805FR-07150RL" H 9850 2200 60  0001 C CNN "Mfg_Part_No"
 	1    9850 2200
 	0    1    1    0

Commit message: Change resistor values use standard ref prefixes
* Fix #1 and #2
Parts:
- removed IC1: ATMEGA328P-A, Housings_QFP:TQFP-32_7x7mm_Pitch0.8mm, symbol ATMEGA328P-A
- added U7: ATMEGA328P-AU, Housings_QFP:TQFP-32_7x7mm_Pitch0.8mm, symbol ATMEGA328P-AU
- FB1, FB2, FB3, FB4: Mfg_Part_No RC0805JR-070RL -> 742792040
- JP1: symbol JUMPER -> Jumper
- renumbered J1 to P7
Changed lines of the file:
@@
 Sheet 1 3
 Title "40-channel HV switching board"
-Date "2017-04-05"
-Rev "3.1"
+Date "2017-06-01"
+Rev "3.1.1"
 Comp "Sci-Bots Inc."
 Comment1 ""
@@
 L LED DS1
 U 1 1 52E82588
-P 2800 1400
-F 0 "DS1" H 2800 1500 50  0000 C CNN
-F 1 "+3.3V_PWR" H 2800 1300 50  0000 C CNN
-F 2 "LEDs:LED_0805" H 2800 1400 60  0001 C CNN
-F 3 "" H 2800 1400 60  0001 C CNN
-F 4 "150080BS75000" H 2800 1400 60  0001 C CNN "Mfg_Part_No"
-	1    2800 1400
+P 2800 1350
+F 0 "DS1" H 2800 1450 50  0000 C CNN
+F 1 "+3.3V_PWR" H 2850 1550 50  0000 C CNN
+F 2 "LEDs:LED_0805" H 2800 1350 60  0001 C CNN
+F 3 "" H 2800 1350 60  0001 C CNN
+F 4 "150080BS75000" H 2800 1350 60  0001 C CNN "Mfg_Part_No"
+	1    2800 1350
 	0    -1   -1   0
 $EndComp
@@
 Text GLabel 9300 3150 2    60   Input ~ 0
 D7
-Text GLabel 2800 1600 2    60   Input ~ 0
+Text GLabel 2800 1500 3    60   Input ~ 0
 GND
 Text GLabel 7050 1150 0    60   Input ~ 0
@@
 	-1   0    0    -1
 $EndComp
-$Comp
-L ATMEGA328P-A IC1
-U 1 1 583628D3
-P 8300 1950
-F 0 "IC1" H 7550 3200 50  0000 L BNN
-F 1 "ATMEGA328P-A" H 8700 550 50  0000 L BNN
-F 2 "Housings_QFP:TQFP-32_7x7mm_Pitch0.8mm" H 8300 500 50  0001 C CIN
-F 3 "" H 8300 1950 50  0000 C CNN
-F 4 "ATMEGA328P-AU" H 8300 1950 60  0001 C CNN "Mfg_Part_No"
-	1    8300 1950
-	1    0    0    -1
-$EndComp
 Text GLabel 9900 1150 2    60   Input ~ 0
 D11/MOSI
@@
 Connection ~ 1950 900
 Wire Wire Line
-	2350 1300 2350 1600
-Wire Wire Line
-	2350 1600 2800 1600
+	2350 1300 2350 1500
+Wire Wire Line
+	2350 1500 2800 1500
 Connection ~ 1950 1300
 $Comp
-L JUMPER JP1
+L Jumper JP1
 U 1 1 58380DDD
 P 900 1950
@@
 D13/SCK
 $Comp
-L TFM-125-02-X-DH J1
+L TFM-125-02-X-DH P7
 U 1 1 58B6BC14
 P 4400 950
-F 0 "J1" H 4600 1100 45  0000 L BNN
+F 0 "P7" H 4600 1100 45  0000 L BNN
 F 1 "TFM-125-02-X-DH" V 4750 -650 45  0000 L BNN
 F 2 "WheelerLab:TFM-125-02-X-DH" H 4430 1100 20  0001 C CNN
@@
 F 2 "Resistors_SMD:R_0805" H 9450 1050 60  0001 C CNN
 F 3 "" H 9450 1050 60  0000 C CNN
-F 4 "RC0805JR-070RL" H 9450 1150 60  0001 C CNN "Mfg_Part_No"
+F 4 "742792040" H 9450 1150 60  0001 C CNN "Mfg_Part_No"
 	1    9450 1150
 	1    0    0    -1
@@
 F 2 "Resistors_SMD:R_0805" H 6000 7550 60  0001 C CNN
 F 3 "" H 6000 7550 60  0000 C CNN
-F 4 "RC0805JR-070RL" H 6000 7650 60  0001 C CNN "Mfg_Part_No"
+F 4 "742792040" H 6000 7650 60  0001 C CNN "Mfg_Part_No"
 	1    6000 7650
 	1    0    0    -1
@@
 F 2 "Resistors_SMD:R_0805" H 9450 1250 60  0001 C CNN
 F 3 "" H 9450 1250 60  0000 C CNN
-F 4 "RC0805JR-070RL" H 9450 1350 60  0001 C CNN "Mfg_Part_No"
+F 4 "742792040" H 9450 1350 60  0001 C CNN "Mfg_Part_No"
 	1    9450 1350
 	1    0    0    -1
@@
 F 2 "Resistors_SMD:R_0805" H 8450 4150 60  0001 C CNN
 F 3 "" H 8450 4150 60  0000 C CNN
-F 4 "RC0805JR-070RL" H 8450 4250 60  0001 C CNN "Mfg_Part_No"
+F 4 "742792040" H 8450 4250 60  0001 C CNN "Mfg_Part_No"
 	1    8450 4250
 	-1   0    0    1
@@
 Wire Wire Line
 	3550 3600 3550 3450
+$Comp
+L ATMEGA328P-AU U7
+U 1 1 59301F62
+P 8300 1950
+F 0 "U7" H 7550 3200 50  0000 L BNN
+F 1 "ATMEGA328P-AU" H 8700 550 50  0000 L BNN
+F 2 "Housings_QFP:TQFP-32_7x7mm_Pitch0.8mm" H 8300 1950 50  0001 C CIN
+F 3 "" H 8300 1950 50  0001 C CNN
+F 4 "ATMEGA328P-AU" H 8300 1950 60  0001 C CNN "Mfg_Part_No"
+	1    8300 1950
+	1    0    0    -1
+$EndComp
 $EndSCHEMATC

Commit message: Modify to use Sci-Bots library submodule
Parts:
- C2, C4: footprint WheelerLab:SM2917 -> Sci-Bots:SM2917
- P7: footprint WheelerLab:TFM-125-02-X-DH -> Sci-Bots:TFM-125-02-X-DH
- U1, U2, U3, U4, U5: footprint WheelerLab:SO16E -> Sci-Bots:SO16E
- Y1: footprint WheelerLab:CSTCE_G15C -> Sci-Bots:CSTCE_G15C
Changed lines of the file:
@@
 LIBS:contrib
 LIBS:valves
-LIBS:wheelerlab
+LIBS:sci-bots
 LIBS:40-channel HV switching board-cache
 EELAYER 25 0
@@
 F 0 "C4" H 1300 1200 50  0000 L CNN
 F 1 "33uF" H 1300 1000 50  0000 L CNN
-F 2 "WheelerLab:SM2917" H 1250 1100 60  0001 C CNN
+F 2 "Sci-Bots:SM2917" H 1250 1100 60  0001 C CNN
 F 3 "" H 1250 1100 60  0001 C CNN
 F 4 "T491D336K020AT" H 1250 1100 60  0001 C CNN "Mfg_Part_No"
@@
 F 0 "C2" H 950 1200 50  0000 L CNN
 F 1 "33uF" H 950 1000 50  0000 L CNN
-F 2 "WheelerLab:SM2917" H 900 1100 60  0001 C CNN
+F 2 "Sci-Bots:SM2917" H 900 1100 60  0001 C CNN
 F 3 "" H 900 1100 60  0001 C CNN
 F 4 "T491D336K020AT" H 900 1100 60  0001 C CNN "Mfg_Part_No"
@@
 F 0 "U1" H 1900 6200 70  0000 C CNN
 F 1 "74HC595A" H 1750 5000 70  0000 C CNN
-F 2 "WheelerLab:SO16E" H 1750 5600 60  0001 C CNN
+F 2 "Sci-Bots:SO16E" H 1750 5600 60  0001 C CNN
 F 3 "~" H 1750 5600 60  0000 C CNN
 F 4 "MM74HC595MX" H 1750 5600 60  0001 C CNN "Mfg_Part_No"
@@
 F 0 "U2" H 4200 6200 70  0000 C CNN
 F 1 "74HC595A" H 4050 5000 70  0000 C CNN
-F 2 "WheelerLab:SO16E" H 4050 5600 60  0001 C CNN
+F 2 "Sci-Bots:SO16E" H 4050 5600 60  0001 C CNN
 F 3 "~" H 4050 5600 60  0000 C CNN
 F 4 "MM74HC595MX" H 4050 5600 60  0001 C CNN "Mfg_Part_No"
@@
 F 0 "U3" H 6550 6200 70  0000 C CNN
 F 1 "74HC595A" H 6400 5000 70  0000 C CNN
-F 2 "WheelerLab:SO16E" H 6400 5600 60  0001 C CNN
+F 2 "Sci-Bots:SO16E" H 6400 5600 60  0001 C CNN
 F 3 "~" H 6400 5600 60  0000 C CNN
 F 4 "MM74HC595MX" H 6400 5600 60  0001 C CNN "Mfg_Part_No"
@@
 F 0 "U4" H 2950 7800 70  0000 C CNN
 F 1 "74HC595A" H 2800 6600 70  0000 C CNN
-F 2 "WheelerLab:SO16E" H 2800 7200 60  0001 C CNN
+F 2 "Sci-Bots:SO16E" H 2800 7200 60  0001 C CNN
 F 3 "~" H 2800 7200 60  0000 C CNN
 F 4 "MM74HC595MX" H 2800 7200 60  0001 C CNN "Mfg_Part_No"
@@
 F 0 "U5" H 5300 7800 70  0000 C CNN
 F 1 "74HC595A" H 5150 6600 70  0000 C CNN
-F 2 "WheelerLab:SO16E" H 5150 7200 60  0001 C CNN
+F 2 "Sci-Bots:SO16E" H 5150 7200 60  0001 C CNN
 F 3 "~" H 5150 7200 60  0000 C CNN
 F 4 "MM74HC595MX" H 5150 7200 60  0001 C CNN "Mfg_Part_No"
@@
 F 0 "Y1" H 9970 1950 60  0000 C CNN
 F 1 "RESONATOR" V 10150 1500 60  0000 C CNN
-F 2 "WheelerLab:CSTCE_G15C" H 9950 1750 60  0001 C CNN
+F 2 "Sci-Bots:CSTCE_G15C" H 9950 1750 60  0001 C CNN
 F 3 "http://www.murata.com/~/media/webrenewal/support/library/catalog/products/timingdevice/ceralock/p16e.ashx" H 9950 1750 60  0001 C CNN
 F 4 "CSTCE8M00G55-R0" H 9950 1750 60  0001 C CNN "Mfg_Part_No"
@@
 F 0 "P7" H 4600 1100 45  0000 L BNN
 F 1 "TFM-125-02-X-DH" V 4750 -650 45  0000 L BNN
-F 2 "WheelerLab:TFM-125-02-X-DH" H 4430 1100 20  0001 C CNN
+F 2 "Sci-Bots:TFM-125-02-X-DH" H 4430 1100 20  0001 C CNN
 F 3 "" H 4400 950 60  0000 C CNN
 F 4 "TFM-125-02-L-DH" H 4400 950 60  0001 C CNN "Mfg_Part_No"
