File: switches_0-19.sch (KiCad schematic (older format))
At the start: 80 parts

Commit message: Change resistor values use standard ref prefixes
* Fix #1 and #2
Parts:
- CH0, CH1, CH10, CH11, CH12, CH13, CH14, CH15, CH16, CH17, CH18, CH19, CH2, CH3, CH4, CH5, CH6, CH8, CH9: value AQW216 -> SSR-DPST; symbol AQW216 -> SSR-DPST; Mfg_Part_No (none) -> TLP227G-2(TP1,N,F)
- CH7: value AQW216 -> SSR-DPST; symbol AQW216 -> SSR-DPST
- R10, R11, R14, R15, R16, R17, R2, R20, R21, R22, R23, R28, R29, R3, R34, R35, R4, R5, R63, R65, R66, R69, R71, R72, R73, R76, R77, R78, R79, R8, R82, R83, R84, R85, R88, R89, R9, R94, R95: value 300 -> 220
- R67: value 300 -> 220; Mfg_Part_No RC0805FR-07300RL -> RC0805FR-07220RL

Commit message: Initial setup with kicad-helpers
Parts:
- R1, R10, R11, R12, R13, R14, R15, R16, R17, R18, R19, R2, R20, R21, R22, R23, R24, R25, R28, R29, R3, R34, R35, R36, R4, R5, R6, R63, R64, R65, R66, R67, R68, R69, R7, R70, R71, R72, R73, R74, R75, R76, R77, R78, R79, R8, R80, R81, R82, R83, R84, R85, R86, R87, R88, R89, R9, R94, R95, R98: symbol R -> Device:R
Changed lines of the file:
@@
-EESchema Schematic File Version 2
-LIBS:power
-LIBS:device
-LIBS:transistors
-LIBS:conn
-LIBS:linear
-LIBS:regul
-LIBS:74xx
-LIBS:cmos4000
-LIBS:adc-dac
-LIBS:memory
-LIBS:xilinx
-LIBS:microcontrollers
-LIBS:dsp
-LIBS:microchip
-LIBS:analog_switches
-LIBS:motorola
-LIBS:texas
-LIBS:intel
-LIBS:audio
-LIBS:interface
-LIBS:digital-audio
-LIBS:philips
-LIBS:display
-LIBS:cypress
-LIBS:siliconi
-LIBS:opto
-LIBS:atmel
-LIBS:contrib
-LIBS:valves
-LIBS:sci-bots
-LIBS:40-channel HV switching board-cache
-EELAYER 25 0
+EESchema Schematic File Version 4
+EELAYER 30 0
 EELAYER END
 $Descr USLetter 11000 8500
@@
 OUT8
 $Comp
-L R R24
+L Device:R R24
 U 1 1 52E6DB5B
 P 3300 1000
@@
 $EndComp
 $Comp
-L R R67
+L Device:R R67
 U 1 1 52E6DB5C
 P 1150 7050
@@
 $EndComp
 $Comp
-L R R73
+L Device:R R73
 U 1 1 52E6DB5E
 P 1150 7750
@@
 $EndComp
 $Comp
-L R R8
+L Device:R R8
 U 1 1 52E6D490
 P 1150 6850
@@
 $EndComp
 $Comp
-L R R2
+L Device:R R2
 U 1 1 52E6DB61
 P 1150 6150
@@
 $EndComp
 $Comp
-L R R65
+L Device:R R65
 U 1 1 52E6DB62
 P 1150 3450
@@
 $EndComp
 $Comp
-L R R71
+L Device:R R71
 U 1 1 52E6D495
 P 1150 4150
@@
 $EndComp
 $Comp
-L R R72
+L Device:R R72
 U 1 1 52E6D496
 P 1150 5950
@@
 $EndComp
 $Comp
-L R R66
+L Device:R R66
 U 1 1 52E6DB67
 P 1150 5250
@@
 $EndComp
 $Comp
-L R R3
+L Device:R R3
 U 1 1 52E6D499
 P 1150 4350
@@
 $EndComp
 $Comp
-L R R9
+L Device:R R9
 U 1 1 52E6DB6A
 P 1150 5050
@@
 $EndComp
 $Comp
-L R R10
+L Device:R R10
 U 1 1 52E6DB6B
 P 1150 3250
@@
 $EndComp
 $Comp
-L R R4
+L Device:R R4
 U 1 1 52E6DB6D
 P 1150 2550
@@
 $EndComp
 $Comp
-L R R63
+L Device:R R63
 U 1 1 52E6DB6E
 P 1150 1650
@@
 HVOUT1
 $Comp
-L R R69
+L Device:R R69
 U 1 1 52E6DB6F
 P 1150 2350
@@
 OUT0
 $Comp
-L R R11
+L Device:R R11
 U 1 1 52E6DB71
 P 1150 1450
@@
 $EndComp
 $Comp
-L R R12
+L Device:R R12
 U 1 1 52E6D4A3
 P 900 1000
@@
 HVOUT0
 $Comp
-L R R5
+L Device:R R5
 U 1 1 52E6DB74
 P 1150 750
@@
 OUT1
 $Comp
-L R R64
+L Device:R R64
 U 1 1 52E6D4A8
 P 900 1900
@@
 	1400 2750 1400 2550
 $Comp
-L R R74
+L Device:R R74
 U 1 1 52E6DB7C
 P 900 2800
@@
 	1400 3650 1400 3450
 $Comp
-L R R1
+L Device:R R1
 U 1 1 52E6DB7F
 P 900 3700
@@
 	1400 4550 1400 4350
 $Comp
-L R R70
+L Device:R R70
 U 1 1 52E6D4B3
 P 900 4600
@@
 	1400 5450 1400 5250
 $Comp
-L R R6
+L Device:R R6
 U 1 1 52E6D4B6
 P 900 5500
@@
 	1400 6350 1400 6150
 $Comp
-L R R7
+L Device:R R7
 U 1 1 52E6D4B9
 P 900 6400
@@
 	1400 7250 1400 7050
 $Comp
-L R R68
+L Device:R R68
 U 1 1 52E6D4BC
 P 900 7300
@@
 $EndComp
 $Comp
-L R R79
+L Device:R R79
 U 1 1 52E6D4C2
 P 3550 7050
@@
 $EndComp
 $Comp
-L R R85
+L Device:R R85
 U 1 1 52E6DB8E
 P 3550 7750
@@
 $EndComp
 $Comp
-L R R20
+L Device:R R20
 U 1 1 52E6DB8F
 P 3550 6850
@@
 $EndComp
 $Comp
-L R R14
+L Device:R R14
 U 1 1 52E6DB91
 P 3550 6150
@@
 $EndComp
 $Comp
-L R R15
+L Device:R R15
 U 1 1 52E6D4E6
 P 3550 4350
@@
 $EndComp
 $Comp
-L R R21
+L Device:R R21
 U 1 1 52E6D4F2
 P 3550 5050
@@
 $EndComp
 $Comp
-L R R84
+L Device:R R84
 U 1 1 52E6D4F8
 P 3550 5950
@@
 $EndComp
 $Comp
-L R R78
+L Device:R R78
 U 1 1 52E6D504
 P 3550 5250
@@
 $EndComp
 $Comp
-L R R16
+L Device:R R16
 U 1 1 52E6DB98
 P 3550 2550
@@
 $EndComp
 $Comp
-L R R22
+L Device:R R22
 U 1 1 52E6D516
 P 3550 3250
@@
 $EndComp
 $Comp
-L R R83
+L Device:R R83
 U 1 1 52E6D51C
 P 3550 4150
@@
 $EndComp
 $Comp
-L R R77
+L Device:R R77
 U 1 1 52E6DB9D
 P 3550 3450
@@
 $EndComp
 $Comp
-L R R76
+L Device:R R76
 U 1 1 52E6D52E
 P 3550 1650
@@
 HVOUT9
 $Comp
-L R R23
+L Device:R R23
 U 1 1 52E6D542
 P 3550 1450
@@
 HVOUT8
 $Comp
-L R R17
+L Device:R R17
 U 1 1 52E6DBA3
 P 3550 750
@@
 OUT9
 $Comp
-L R R75
+L Device:R R75
 U 1 1 52E6D572
 P 3300 1900
@@
 	3800 2750 3800 2550
 $Comp
-L R R86
+L Device:R R86
 U 1 1 52E6D5A6
 P 3300 2800
@@
 	3800 3650 3800 3450
 $Comp
-L R R13
+L Device:R R13
 U 1 1 52E6D5C4
 P 3300 3700
@@
 	3800 4550 3800 4350
 $Comp
-L R R81
+L Device:R R81
 U 1 1 52E6D5E2
 P 3300 4600
@@
 	3800 5450 3800 5250
 $Comp
-L R R18
+L Device:R R18
 U 1 1 52E6D600
 P 3300 5500
@@
 	3800 6350 3800 6150
 $Comp
-L R R19
+L Device:R R19
 U 1 1 52E6DBB7
 P 3300 6400
@@
 	3800 7250 3800 7050
 $Comp
-L R R80
+L Device:R R80
 U 1 1 52E6D63C
 P 3300 7300
@@
 OUT16
 $Comp
-L R R36
+L Device:R R36
 U 1 1 52E6D80A
 P 5700 1000
@@
 $EndComp
 $Comp
-L R R28
+L Device:R R28
 U 1 1 52E6D858
 P 5950 2550
@@
 $EndComp
 $Comp
-L R R34
+L Device:R R34
 U 1 1 52E6D864
 P 5950 3250
@@
 $EndComp
 $Comp
-L R R95
+L Device:R R95
 U 1 1 52E6D86A
 P 5950 4150
@@
 $EndComp
 $Comp
-L R R89
+L Device:R R89
 U 1 1 52E6DBC1
 P 5950 3450
@@
 $EndComp
 $Comp
-L R R88
+L Device:R R88
 U 1 1 52E6D87C
 P 5950 1650
@@
 HVOUT17
 $Comp
-L R R94
+L Device:R R94
 U 1 1 52E6D883
 P 5950 2350
@@
 $EndComp
 $Comp
-L R R35
+L Device:R R35
 U 1 1 52E6D88F
 P 5950 1450
@@
 HVOUT16
 $Comp
-L R R29
+L Device:R R29
 U 1 1 52E6D89E
 P 5950 750
@@
 OUT17
 $Comp
-L R R87
+L Device:R R87
 U 1 1 52E6DBCA
 P 5700 1900
@@
 	6200 2750 6200 2550
 $Comp
-L R R98
+L Device:R R98
 U 1 1 52E6DBCF
 P 5700 2800
@@
 	6200 3650 6200 3450
 $Comp
-L R R25
+L Device:R R25
 U 1 1 52E6D90B
 P 5700 3700
@@
 GND
 $Comp
-L R R82
+L Device:R R82
 U 1 1 52E6D535
 P 3550 2350

Commit message: Fix broken symbols
Parts:
- CH0, CH1, CH10, CH11, CH12, CH13, CH14, CH15, CH16, CH17, CH18, CH19, CH2, CH3, CH4, CH5, CH6, CH7, CH8, CH9: value SSR-DPST -> AQW214; symbol SSR-DPST -> sci-bots:AQW214
Connections:
- wire segments 260 -> 280

Commit message: Fix BOM
Parts:
- CH0, CH1, CH10, CH11, CH12, CH13, CH14, CH15, CH16, CH17, CH18, CH19, CH2, CH3, CH4, CH5, CH6, CH7, CH8, CH9: MPN (none) -> AQW214EAZ; Manufacturer (none) -> Panasonic; Mfg_Part_No TLP227G-2(TP1,N,F) -> (none)
- R1, R12, R13, R18, R19, R25, R36, R6, R64, R68, R7, R70, R74, R75, R80, R81, R86, R87, R98: MPN (none) -> RC0805FR-074K75L; Manufacturer (none) -> Yageo
- R10, R11, R14, R15, R16, R17, R2, R20, R21, R22, R23, R28, R29, R3, R34, R35, R4, R5, R63, R65, R66, R69, R71, R72, R73, R76, R77, R78, R79, R8, R82, R83, R84, R85, R88, R89, R9, R94, R95: MPN (none) -> RC0805FR-07220RL; Manufacturer (none) -> Yageo
- R24: MPN (none) -> RC0805FR-074K75L; Manufacturer (none) -> Yageo; Mfg_Part_No RC0805FR-074K75L -> (none)
- R67: MPN (none) -> RC0805FR-07220RL; Manufacturer (none) -> Yageo; Mfg_Part_No RC0805FR-07220RL -> (none)
