File: 40-channel-hv-switching-board.sch (KiCad schematic (older format))
At the start: 44 parts, among them P1 CONN_01X06, P2 CONN_01X06, P3 CONN_01X01, P4 CONN_01X01, P5 CONN_01X01, P6 CONN_01X01, P7 TFM-125-02-X-DH, U1 74HC595A, U2 74HC595A, U3 74HC595A, U4 74HC595A, U5 74HC595A, U6 W25Q64FV, U7 ATMEGA328P-AU, Y1 RESONATOR

Commit message: Fix broken symbols
Parts:
- U7: symbol ATMEGA328P-AU -> MCU_Microchip_ATmega:ATmega328P-AU
Connections:
- wire segments 84 -> 81
Other:
- moved on the sheet: C10, C11, C13, C14, C15, FB1, FB3, FB4, R100, R125, R126, R99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

Commit message: Get all tests passing
Parts:
- JP1, P1, P2, P3, P4, P5, P6: MPN (none) -> DNP; Manufacturer (none) -> DNP
Connections:
- net +3.3V: now also P2.5 (Pin_5)
- net CHASIS_GND: now also P4.1 (Pin_1), P5.1 (Pin_1)
- net D11/MOSI: now also P2.3 (Pin_3)
- net D12/MISO: now also P2.6 (Pin_6)
- net D13/SCK: now also P2.4 (Pin_4)
- net GND: now also P2.1 (Pin_1)
- net RST: now also P2.2 (Pin_2)
- net D10/SS: no longer names the net of U7.14 (PB2)
- net D7: no longer names the net of U7.11 (PD7)
- no-connect marks 10 -> 13
