File: 40-channel-hv-switching-board.kicad_pcb (KiCad board)
At the start: 4 copper layers, 84 x 92 mm, 207 parts, among them P1 CONN_01X06, P2 CONN_01X06, P3 CONN_01X01, P4 CONN_01X01, P5 CONN_01X01, P6 CONN_01X01, P7 TFM-125-02-X-DH, U1 74HC595A, U2 74HC595A, U3 74HC595A, U4 74HC595A, U5 74HC595A, U6 W25Q64FV, U7 ATMEGA328P-AU, Y1 RESONATOR

Commit message: Get all tests passing
Parts:
- CH0, CH1, CH10, CH11, CH12, CH13, CH14, CH15, CH16, CH17, CH18, CH19, CH2, CH20, CH21, CH22, CH23, CH24, CH25, CH26, CH27, CH28, CH29, CH3, CH30, CH31, CH32, CH33, CH34, CH35, CH36, CH37, CH38, CH39, CH4, CH5, CH6, CH7, CH8, CH9: value SSR-DPST -> AQW214
Connections:
- net D10/SS renamed Net-(U7-Pad14)
- net D7 renamed Net-(U7-Pad11)

Commit message: Update netlist
Parts:
- removed G***: LOGO, LOGO
- removed G***: LOGO, Sci-Bots:OSHW_logo_10mm
- removed G***: LOGO, Sci-Bots:CC_S_A_logo_10mm
